File: KiCad/DIB_interface.kicad_sch (KiCad schematic)
At the start: 30 parts, among them IC1 USB3300-EZK, IC2 M24C32-DFDW6TP, IC3 ISO6762FDWR, IC4 ISO6762FDWR, IC5 ISO6762FDWR, X2 CBED202-1379B001C1AD

Commit message: Gerber files added
Parts:
- X2: DigiKey (none) -> 4217-CBED202-1379B001C1ADCT-ND; LCSC (none) -> C5611301; TME (none) -> -
Changed lines of the file:
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@@
 			)
 		)
-		(property "DigiKey" ""
+		(property "DigiKey" "4217-CBED202-1379B001C1ADCT-ND"
 			(at 111.76 63.5 0)
 			(hide yes)
@@
 			)
 		)
-		(property "TME" ""
+		(property "TME" "-"
 			(at 111.76 68.58 0)
 			(hide yes)
@@
 			)
 		)
-		(property "LCSC" ""
+		(property "LCSC" "C5611301"
 			(at 111.76 71.12 0)
 			(hide yes)

Commit message: BOM update
Parts:
- R1, R2: DigiKey (none) -> 13-AC0603FR-0715RLCT-ND; LCSC (none) -> C144698; Mouser (none) -> 603-AC0603FR-0715RL; TME (none) -> CQ0603-15R-1%
- R5: DigiKey (none) -> 13-AC0603FR-7W470RLCT-ND; LCSC (none) -> C20142029; Mouser (none) -> 603-AC0603FR-7W470RL; TME (none) -> SMD0603-470R-1%
- RN1, RN2: value CAY16A-XXX -> CAY16-330J4LF; LCSC (none) -> C840641
Changed lines of the file:
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@@
 	(title_block
 		(title "${project_name}")
-		(date "2026-07-24")
+		(date "2026-07-25")
 		(rev "${project_version}")
 		(company "${project_creator}")
@@
 			)
 		)
-		(property "Value" "CAY16A-XXX"
+		(property "Value" "CAY16-330J4LF"
 			(at 254 50.8 0)
 			(show_name no)
@@
 			)
 		)
-		(property "LCSC" ""
+		(property "LCSC" "C840641"
 			(at 254 48.26 0)
 			(hide yes)
@@
 			)
 		)
-		(property "DigiKey" ""
+		(property "DigiKey" "13-AC0603FR-0715RLCT-ND"
 			(at 78.74 134.62 0)
 			(hide yes)
@@
 			)
 		)
-		(property "Mouser" ""
+		(property "Mouser" "603-AC0603FR-0715RL"
 			(at 78.74 134.62 0)
 			(hide yes)
@@
 			)
 		)
-		(property "TME" ""
+		(property "TME" "CQ0603-15R-1%"
 			(at 78.74 134.62 0)
 			(hide yes)
@@
 			)
 		)
-		(property "LCSC" ""
+		(property "LCSC" "C144698"
 			(at 78.74 134.62 0)
 			(hide yes)
@@
 			)
 		)
-		(property "Value" "CAY16A-XXX"
+		(property "Value" "CAY16-330J4LF"
 			(at 35.56 83.82 0)
 			(hide yes)
@@
 			)
 		)
-		(property "LCSC" ""
+		(property "LCSC" "C840641"
 			(at 35.56 81.28 0)
 			(hide yes)
@@
 			)
 		)
-		(property "DigiKey" ""
+		(property "DigiKey" "13-AC0603FR-7W470RLCT-ND"
 			(at 127 137.16 0)
 			(hide yes)
@@
 			)
 		)
-		(property "Mouser" ""
+		(property "Mouser" "603-AC0603FR-7W470RL"
 			(at 127 137.16 0)
 			(hide yes)
@@
 			)
 		)
-		(property "TME" ""
+		(property "TME" "SMD0603-470R-1%"
 			(at 127 137.16 0)
 			(hide yes)
@@
 			)
 		)
+		(property "LCSC" "C20142029"
+			(at 127 137.16 90)
+			(hide yes)
+			(show_name no)
+			(do_not_autoplace no)
+			(effects
+				(font
+					(size 0.889 0.889)
+				)
+			)
+		)
 		(pin "1"
 		)
@@
 			)
 		)
-		(property "Value" "CAY16A-XXX"
+		(property "Value" "CAY16-330J4LF"
 			(at 35.56 88.9 0)
 			(hide yes)
@@
 			)
 		)
-		(property "LCSC" ""
+		(property "LCSC" "C840641"
 			(at 35.56 86.36 0)
 			(hide yes)
@@
 			)
 		)
-		(property "DigiKey" ""
+		(property "DigiKey" "13-AC0603FR-0715RLCT-ND"
 			(at 78.74 165.1 0)
 			(hide yes)
@@
 			)
 		)
-		(property "Mouser" ""
+		(property "Mouser" "603-AC0603FR-0715RL"
 			(at 78.74 165.1 0)
 			(hide yes)
@@
 			)
 		)
-		(property "TME" ""
+		(property "TME" "CQ0603-15R-1%"
 			(at 78.74 165.1 0)
 			(hide yes)
@@
 			)
 		)
-		(property "LCSC" ""
+		(property "LCSC" "C144698"
 			(at 78.74 165.1 0)
 			(hide yes)
@@
 			)
 		)
-		(property "Value" "CAY16A-XXX"
+		(property "Value" "CAY16-330J4LF"
 			(at 254 45.72 0)
 			(hide yes)
@@
 			)
 		)
-		(property "LCSC" ""
+		(property "LCSC" "C840641"
 			(at 254 43.18 0)
 			(hide yes)
@@
 			)
 		)
-		(property "Value" "CAY16A-XXX"
+		(property "Value" "CAY16-330J4LF"
 			(at 35.56 86.36 0)
 			(hide yes)
@@
 			)
 		)
-		(property "LCSC" ""
+		(property "LCSC" "C840641"
 			(at 35.56 83.82 0)
 			(hide yes)
@@
 			)
 		)
-		(property "Value" "CAY16A-XXX"
+		(property "Value" "CAY16-330J4LF"
 			(at 254 48.26 0)
 			(hide yes)
@@
 			)
 		)
-		(property "LCSC" ""
+		(property "LCSC" "C840641"
 			(at 254 45.72 0)
 			(hide yes)
@@
 			)
 		)
-		(property "Value" "CAY16A-XXX"
+		(property "Value" "CAY16-330J4LF"
 			(at 35.56 92.71 0)
 			(show_name no)
@@
 			)
 		)
-		(property "LCSC" ""
+		(property "LCSC" "C840641"
 			(at 35.56 91.44 0)
 			(hide yes)
@@
 			)
 		)
-		(property "Value" "CAY16A-XXX"
+		(property "Value" "CAY16-330J4LF"
 			(at 254 43.18 0)
 			(hide yes)
@@
 			)
 		)
-		(property "LCSC" ""
+		(property "LCSC" "C840641"
 			(at 254 40.64 0)
 			(hide yes)
