File: KiCad/DIB_interface.kicad_sch (KiCad schematic)
At the start: 30 parts, among them IC1 USB3300-EZK, IC2 M24C32-DFDW6TP, IC3 ISO6762FDWR, IC4 ISO6762FDWR, IC5 ISO6762FDWR, X2 CBED202-1379B001C1AD

Commit message: Image of assembled prototype
Parts:
- added TP9: Test, PCM_EEZ_THT:TEST-5, symbol PCM_EEZ_unsorted:PCB test point
- C4, C6, C8: value 4u7 -> 4u7/35V; DigiKey 1276-1044-1-ND -> 1276-6794-1-ND; LCSC C19666 -> C913498; Mouser 187-CL10A475KP8NNNC -> 81-GRM188R6YA475ME5D; TME CL10A475KP8NNNC -> GRM219R6YA475KA73D
Connections:
- net GND: now also TP9.1 (P$1)
Changed lines of the file:
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@@
 	(title_block
 		(title "${project_name}")
-		(date "2026-08-25")
+		(date "2026-08-30")
 		(rev "${project_version}")
 		(company "${project_creator}")
@@
 			)
 		)
-		(property "Value" "4u7"
+		(property "Value" "4u7/35V"
 			(at 132.08 184.15 0)
 			(show_name no)
@@
 			)
 		)
-		(property "DigiKey" "1276-1044-1-ND"
+		(property "DigiKey" "1276-6794-1-ND"
 			(at 132.08 180.34 0)
 			(hide yes)
@@
 			)
 		)
-		(property "Mouser" "187-CL10A475KP8NNNC"
+		(property "Mouser" "81-GRM188R6YA475ME5D"
 			(at 132.08 180.34 0)
 			(hide yes)
@@
 			)
 		)
-		(property "TME" "CL10A475KP8NNNC"
+		(property "TME" "GRM219R6YA475KA73D"
 			(at 132.08 180.34 0)
 			(hide yes)
@@
 			)
 		)
-		(property "LCSC" "C19666"
+		(property "LCSC" "C913498"
 			(at 132.08 180.34 0)
 			(hide yes)
@@
 	)
 	(symbol
+		(lib_id "PCM_EEZ_unsorted:PCB test point")
+		(at 35.56 53.34 0)
+		(mirror y)
+		(unit 1)
+		(body_style 1)
+		(exclude_from_sim no)
+		(in_bom no)
+		(on_board yes)
+		(in_pos_files no)
+		(dnp no)
+		(property "Reference" "TP9"
+			(at 33.655 53.34 0)
+			(show_name no)
+			(do_not_autoplace no)
+			(effects
+				(font
+					(size 1.27 1.27)
+				)
+				(justify left)
+			)
+		)
+		(property "Value" "Test"
+			(at 35.56 55.88 0)
+			(hide yes)
+			(show_name no)
+			(do_not_autoplace no)
+			(effects
+				(font
+					(size 1.27 1.27)
+				)
+				(justify left bottom)
+			)
+		)
+		(property "Footprint" "PCM_EEZ_THT:TEST-5"
+			(at 35.56 55.88 0)
+			(hide yes)
+			(show_name no)
+			(do_not_autoplace no)
+			(effects
+				(font
+					(size 1.27 1.27)
+				)
+			)
+		)
+		(property "Datasheet" ""
+			(at 35.56 53.34 0)
+			(hide yes)
+			(show_name no)
+			(do_not_autoplace no)
+			(effects
+				(font
+					(size 1.27 1.27)
+				)
+			)
+		)
+		(property "Description" ""
+			(at 35.56 53.34 0)
+			(hide yes)
+			(show_name no)
+			(do_not_autoplace no)
+			(effects
+				(font
+					(size 1.27 1.27)
+				)
+			)
+		)
+		(property "DigiKey" ""
+			(at 35.56 53.34 0)
+			(hide yes)
+			(show_name no)
+			(do_not_autoplace no)
+			(effects
+				(font
+					(size 0.889 0.889)
+				)
+			)
+		)
+		(property "Mouser" ""
+			(at 35.56 53.34 0)
+			(hide yes)
+			(show_name no)
+			(do_not_autoplace no)
+			(effects
+				(font
+					(size 0.889 0.889)
+				)
+			)
+		)
+		(property "TME" ""
+			(at 35.56 53.34 0)
+			(hide yes)
+			(show_name no)
+			(do_not_autoplace no)
+			(effects
+				(font
+					(size 0.889 0.889)
+				)
+			)
+		)
+		(property "LCSC" ""
+			(at 35.56 53.34 0)
+			(hide yes)
+			(show_name no)
+			(do_not_autoplace no)
+			(effects
+				(font
+					(size 0.889 0.889)
+				)
+			)
+		)
+		(property "Label" "GND"
+			(at 35.56 53.34 0)
+			(hide yes)
+			(show_name no)
+			(do_not_autoplace no)
+			(effects
+				(font
+					(size 0.889 0.889)
+				)
+			)
+		)
+		(pin "1"
+		)
+		(instances
+			(project "EEZ DIB MIO168plus"
+				(path "/8165d74e-be16-4c9d-8240-91910dc4b43e/a09a6849-987f-46b9-b52e-df6cf57fd371"
+					(reference "TP9")
+					(unit 1)
+				)
+			)
+		)
+	)
+	(symbol
 		(lib_id "PCM_EEZ_symbols:+3V3_ISO")
 		(at 248.92 76.2 0)
@@
 			)
 		)
-		(property "Value" "4u7"
+		(property "Value" "4u7/35V"
 			(at 142.24 184.15 0)
 			(show_name no)
@@
 			)
 		)
-		(property "DigiKey" "1276-1044-1-ND"
+		(property "DigiKey" "1276-6794-1-ND"
 			(at 142.24 180.34 0)
 			(hide yes)
@@
 			)
 		)
-		(property "Mouser" "187-CL10A475KP8NNNC"
+		(property "Mouser" "81-GRM188R6YA475ME5D"
 			(at 142.24 180.34 0)
 			(hide yes)
@@
 			)
 		)
-		(property "TME" "CL10A475KP8NNNC"
+		(property "TME" "GRM219R6YA475KA73D"
 			(at 142.24 180.34 0)
 			(hide yes)
@@
 			)
 		)
-		(property "LCSC" "C19666"
+		(property "LCSC" "C913498"
 			(at 142.24 180.34 0)
 			(hide yes)
@@
 			)
 		)
-		(property "Value" "4u7"
+		(property "Value" "4u7/35V"
 			(at 137.16 184.15 0)
 			(show_name no)
@@
 			)
 		)
-		(property "DigiKey" "1276-1044-1-ND"
+		(property "DigiKey" "1276-6794-1-ND"
 			(at 137.16 180.34 0)
 			(hide yes)
@@
 			)
 		)
-		(property "Mouser" "187-CL10A475KP8NNNC"
+		(property "Mouser" "81-GRM188R6YA475ME5D"
 			(at 137.16 180.34 0)
 			(hide yes)
@@
 			)
 		)
-		(property "TME" "CL10A475KP8NNNC"
+		(property "TME" "GRM219R6YA475KA73D"
 			(at 137.16 180.34 0)
 			(hide yes)
@@
 			)
 		)
-		(property "LCSC" "C19666"
+		(property "LCSC" "C913498"
 			(at 137.16 180.34 0)
 			(hide yes)

Commit message: BOM updated
Other:
- moved on the sheet: C6, C8
Changed lines of the file:
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@@
 	)
 	(junction
-		(at 142.24 185.42)
+		(at 147.32 185.42)
 		(diameter 0)
 		(color 0 0 0 0)
@@
 	(wire
 		(pts
-			(xy 137.16 185.42) (xy 142.24 185.42)
+			(xy 139.7 185.42) (xy 147.32 185.42)
 		)
 		(stroke
@@
 	(wire
 		(pts
-			(xy 142.24 172.72) (xy 142.24 177.8)
+			(xy 147.32 172.72) (xy 147.32 177.8)
 		)
 		(stroke
@@
 	(wire
 		(pts
-			(xy 119.38 172.72) (xy 142.24 172.72)
+			(xy 119.38 172.72) (xy 147.32 172.72)
 		)
 		(stroke
@@
 	(wire
 		(pts
-			(xy 119.38 175.26) (xy 137.16 175.26)
+			(xy 119.38 175.26) (xy 139.7 175.26)
 		)
 		(stroke
@@
 	(wire
 		(pts
-			(xy 137.16 175.26) (xy 137.16 177.8)
+			(xy 139.7 175.26) (xy 139.7 177.8)
 		)
 		(stroke
@@
 	(symbol
 		(lib_id "PCM_EEZ_symbols:GND")
-		(at 142.24 187.96 0)
+		(at 147.32 187.96 0)
 		(unit 1)
 		(body_style 1)
@@
 		(dnp no)
 		(property "Reference" "#GND09"
-			(at 142.24 187.96 0)
+			(at 147.32 187.96 0)
 			(hide yes)
 			(show_name no)
@@
 		)
 		(property "Value" "GND"
-			(at 142.24 189.865 0)
+			(at 147.32 189.865 0)
 			(show_name no)
 			(do_not_autoplace no)
@@
 		)
 		(property "Footprint" ""
-			(at 142.24 187.96 0)
+			(at 147.32 187.96 0)
 			(hide yes)
 			(show_name no)
@@
 		)
 		(property "Datasheet" ""
-			(at 142.24 187.96 0)
+			(at 147.32 187.96 0)
 			(hide yes)
 			(show_name no)
@@
 		)
 		(property "Description" ""
-			(at 142.24 187.96 0)
+			(at 147.32 187.96 0)
 			(hide yes)
 			(show_name no)
@@
 			(effects
 				(font
-					(size 1.27 1.27)
+					(size 1.016 1.016)
 				)
 				(justify right bottom)
@@
 	(symbol
 		(lib_id "PCM_EEZ_passives:C-EU")
-		(at 142.24 180.34 0)
+		(at 147.32 180.34 0)
 		(mirror y)
 		(unit 1)
@@
 		(dnp no)
 		(property "Reference" "C8"
-			(at 142.24 180.34 0)
+			(at 147.32 180.34 0)
 			(show_name no)
 			(do_not_autoplace no)
@@
 		)
 		(property "Value" "4u7/35V"
-			(at 142.24 184.15 0)
+			(at 147.32 184.15 0)
 			(show_name no)
 			(do_not_autoplace no)
 			(effects
 				(font
-					(size 1.27 1.27)
+					(size 1.016 1.016)
 				)
 				(justify right bottom)
@@
 		)
 		(property "Footprint" "PCM_EEZ_passives:C_0603_1608Metric"
-			(at 142.24 177.8 0)
+			(at 147.32 177.8 0)
 			(hide yes)
 			(show_name no)
@@
 		)
 		(property "Datasheet" ""
-			(at 142.24 177.8 0)
+			(at 147.32 177.8 0)
 			(hide yes)
 			(show_name no)
@@
 		)
 		(property "Description" ""
-			(at 142.24 180.34 90)
+			(at 147.32 180.34 90)
 			(hide yes)
 			(show_name no)
@@
 		)
 		(property "DigiKey" "1276-6794-1-ND"
-			(at 142.24 180.34 0)
+			(at 147.32 180.34 0)
 			(hide yes)
 			(show_name no)
@@
 		)
 		(property "Mouser" "81-GRM188R6YA475ME5D"
-			(at 142.24 180.34 0)
+			(at 147.32 180.34 0)
 			(hide yes)
 			(show_name no)
@@
 		)
 		(property "TME" "GRM219R6YA475KA73D"
-			(at 142.24 180.34 0)
+			(at 147.32 180.34 0)
 			(hide yes)
 			(show_name no)
@@
 		)
 		(property "LCSC" "C913498"
-			(at 142.24 180.34 0)
+			(at 147.32 180.34 0)
 			(hide yes)
 			(show_name no)
@@
 		)
 		(property "Comment" ""
-			(at 142.24 180.34 0)
+			(at 147.32 180.34 0)
 			(hide yes)
 			(show_name no)
@@
 	(symbol
 		(lib_id "PCM_EEZ_passives:C-EU")
-		(at 137.16 180.34 0)
+		(at 139.7 180.34 0)
 		(mirror y)
 		(unit 1)
@@
 		(dnp no)
 		(property "Reference" "C6"
-			(at 137.16 180.34 0)
+			(at 139.7 180.34 0)
 			(show_name no)
 			(do_not_autoplace no)
@@
 		)
 		(property "Value" "4u7/35V"
-			(at 137.16 184.15 0)
+			(at 139.7 184.15 0)
 			(show_name no)
 			(do_not_autoplace no)
 			(effects
 				(font
-					(size 1.27 1.27)
+					(size 1.016 1.016)
 				)
 				(justify right bottom)
@@
 		)
 		(property "Footprint" "PCM_EEZ_passives:C_0603_1608Metric"
-			(at 137.16 177.8 0)
+			(at 139.7 177.8 0)
 			(hide yes)
 			(show_name no)
@@
 		)
 		(property "Datasheet" ""
-			(at 137.16 177.8 0)
+			(at 139.7 177.8 0)
 			(hide yes)
 			(show_name no)
@@
 		)
 		(property "Description" ""
-			(at 137.16 180.34 90)
+			(at 139.7 180.34 90)
 			(hide yes)
 			(show_name no)
@@
 		)
 		(property "DigiKey" "1276-6794-1-ND"
-			(at 137.16 180.34 0)
+			(at 139.7 180.34 0)
 			(hide yes)
 			(show_name no)
@@
 		)
 		(property "Mouser" "81-GRM188R6YA475ME5D"
-			(at 137.16 180.34 0)
+			(at 139.7 180.34 0)
 			(hide yes)
 			(show_name no)
@@
 		)
 		(property "TME" "GRM219R6YA475KA73D"
-			(at 137.16 180.34 0)
+			(at 139.7 180.34 0)
 			(hide yes)
 			(show_name no)
@@
 		)
 		(property "LCSC" "C913498"
-			(at 137.16 180.34 0)
+			(at 139.7 180.34 0)
 			(hide yes)
 			(show_name no)
@@
 		)
 		(property "Comment" ""
-			(at 137.16 180.34 0)
+			(at 139.7 180.34 0)
 			(hide yes)
 			(show_name no)

Commit message: DIB_SYNC added to isolator (currently not used)
Connections:
- net DIB_OE_SYNC is gone; now on net DIB_SYNC: X1.B13 (OE_SNYC)
- net DIB_SYNC: now reaches IC4.2 (INA)
- no-connect marks 44 -> 43
Changed lines of the file:
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@@
 	(title_block
 		(title "${project_name}")
-		(date "2026-09-19")
+		(date "2026-09-21")
 		(rev "${project_version}")
 		(company "${project_creator}")
@@
 	)
 	(no_connect
-		(at 246.38 88.9)
-	)
-	(no_connect
 		(at 43.18 60.96)
 	)
@@
 	)
 	(no_connect
+		(at 246.38 88.9)
+	)
+	(no_connect
 		(at 43.18 33.02)
 	)
@@
 	)
 	(no_connect
-		(at 210.82 88.9)
-	)
-	(no_connect
 		(at 43.18 50.8)
 	)
@@
 	(wire
 		(pts
+			(xy 205.74 88.9) (xy 210.82 88.9)
+		)
+		(stroke
+			(width 0)
+			(type default)
+		)
+	)
+	(wire
+		(pts
 			(xy 200.66 30.48) (xy 200.66 33.02)
 		)
@@
 		)
 	)
-	(global_label "DIB_OE_SYNC"
+	(global_label "DIB_SYNC"
 		(shape output)
 		(at 76.2 60.96 0)
@@
 			)
 		)
+	)
+	(global_label "DIB_SYNC"
+		(shape input)
+		(at 205.74 88.9 180)
+		(fields_autoplaced yes)
+		(effects
+			(font
+				(size 0.889 0.889)
+			)
+			(justify right)
+		)
+		(property "Intersheetrefs" "${INTERSHEET_REFS}"
+			(at 194.93 88.9 0)
+			(hide yes)
+			(show_name no)
+			(do_not_autoplace no)
+			(effects
+				(font
+					(size 1.27 1.27)
+				)
+				(justify right)
+			)
+		)
