File: KiCad/DIB_interface.kicad_sch (KiCad schematic)
At the start: 31 parts, among them IC1 USB3300-EZK, IC2 M24C32-DFDW6TP, IC3 ISO6762FDWR, IC4 ISO6762FDWR, IC5 ISO6762FDWR, X2 CBED202-1379B001C1AD

Commit message: Gerbers updated
Parts:
- X1: now in the parts list
Connections:
- net CLK_IN: now reaches X1.B17 (REFCLK+)
- no-connect marks 43 -> 42
Changed lines of the file:
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@@
 	(title_block
 		(title "${project_name}")
-		(date "2026-09-21")
+		(date "2026-10-08")
 		(rev "${project_version}")
 		(company "${project_creator}")
@@
 	)
 	(no_connect
-		(at 71.12 71.12)
-	)
-	(no_connect
 		(at 71.12 93.98)
 	)
@@
 	(wire
 		(pts
+			(xy 76.2 71.12) (xy 71.12 71.12)
+		)
+		(stroke
+			(width 0)
+			(type default)
+		)
+	)
+	(wire
+		(pts
 			(xy 248.92 127) (xy 251.46 127)
 		)
@@
 		)
 	)
+	(global_label "CLK_IN"
+		(shape output)
+		(at 76.2 71.12 0)
+		(fields_autoplaced yes)
+		(effects
+			(font
+				(size 0.889 0.889)
+			)
+			(justify left)
+		)
+		(property "Intersheetrefs" "${INTERSHEET_REFS}"
+			(at 82.8191 71.12 0)
+			(hide yes)
+			(show_name no)
+			(do_not_autoplace no)
+			(effects
+				(font
+					(size 1.27 1.27)
+				)
+				(justify left)
+			)
+		)
+	)
 	(global_label "I2C_SDA"
 		(shape bidirectional)
@@
 		(body_style 1)
 		(exclude_from_sim no)
-		(in_bom no)
+		(in_bom yes)
 		(on_board yes)
 		(in_pos_files yes)

Commit message: #4
Parts:
- added C1: 100n, PCM_EEZ_passives:C_0603_1608Metric, symbol PCM_EEZ_passives:C-EU
- added IC1: SN74LVC1G126DBVR, PCM_EEZ_SMD:DBV5, symbol PCM_EEZ_TI:SN74LVC1G126
- added R3: 10K, PCM_EEZ_passives:R_0603_1608Metric, symbol PCM_EEZ_passives:R-EU
- renumbered C9 to C10, C10 to C11, C11 to C12, C12 to C13, C13 to C14, C14 to C15, C15 to C16, C1 to C2, C2 to C3, C3 to C4, C4 to C5, C5 to C6, C6 to C7, C7 to C8, C8 to C9, IC1 to IC2, IC2 to IC3, IC3 to IC4, IC4 to IC5, IC5 to IC6, R5 to R4, R6 to R5, R3 to R6, R4 to R7, TP9 to TP1
Connections:
- net +3V3: now also C1.1, IC1.5 (VCC), R3.2
- net DIB_BOOT0: now also IC1.1 (OE)
- net GND: now also C1.2, IC1.3 (GND)
- net DIB_TOUT: now reaches X1.B15 (TOUT)
- net DIB_UART_RX: now reaches X1.B18 (UART_RX)
- net DIB_UART_RX: now also IC1.4 (Y)
- net UART_RX: now reaches X1.B19 (UART_TX)
- new net UART_TX: IC1.2 (A), R3.1
- no-connect marks 42 -> 39
Other:
- moved on the sheet: C10, C11, C12, C13, C14, C15, C16, IC3, IC5, IC6, R6, R7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
