File: KiCad/EEZ DIB MIO168plus.kicad_pcb (KiCad board)
At the start: 4 copper layers, 191 x 95 mm, 273 parts, among them IC1 USB3300-EZK, IC10 L78L15, IC11 L79L15, IC12 74HC126PW,118, IC13 OPA2196IDR, IC14 DAC7760IPWPR, IC15 DAC7760IPWPR, IC16 SN74LVC138ADBR, IC17 DAC7563TDGSR, IC18 OPA376AIDBVR, IC19 PCAL9714HNMP, IC2 M24C32-DFDW6TP, IC20 OPA2196IDR, IC21 TLE75008ESDXUMA1, IC22 TL431B, IC3 ISO6762FDWR, IC4 ISO6762FDWR, IC5 ISO6762FDWR, IC6 STM32F446ZET6, IC7 IS42S16400N-6TL, IC8 SN6505BDBVT, IC9 TPS7A2033PDBVR, Q1 MMBT5401, Q10 2N7002PS,115, Q11 2N7002PS,115, Q2 MMBT5551, Q3 MMBT5551, Q4 IRLML2246TRPBF, Q5 2N7002, Q6 IRLML2246TRPBF, Q7 2N7002PS,115, Q8 2N7002PS,115, Q9 2N7002PS,115, X2 CBED202-1379B001C1AD, X4 1844824, Y1 LF XTAL026392

Commit message: Gerbers updated
Parts:
- TP4: footprint PCM_EEZ_THT:Testhole 24_50mils -> PCM_EEZ_THT:TEST-5
- moved TP4 0.61 mm to (185.4, 120.6)
Changed lines of the file:
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@@
 		(filling no)
 		(pcbplotparams
-			(layerselection 0x00000000_00000000_55555555_5755f5ff)
+			(layerselection 0x00000000_00000000_555555d5_5755f5ff)
 			(plot_on_all_layers_selection 0x00000000_00000000_00000000_00000000)
 			(disableapertmacros no)
@@
 		)
 	)
-	(footprint "PCM_EEZ_THT:Testhole 24_50mils"
+	(footprint "PCM_EEZ_THT:TEST-5"
 		(layer "F.Cu")
-		(at 185.377738 121.24)
+		(at 185.377738 120.63)
 		(property "Reference" "TP4"
-			(at 0.01 -1.21 0)
+			(at -1.147738 -1.42 0)
 			(unlocked yes)
 			(layer "F.SilkS")
@@
 					(bold yes)
 				)
+				(justify left)
 			)
 		)
 		(property "Value" "Test"
-			(at 0 1 0)
+			(at 0 0 0)
 			(unlocked yes)
 			(layer "F.Fab")
 			(effects
 				(font
-					(size 1 1)
-					(thickness 0.15)
+					(size 0.6096 0.6096)
+					(thickness 0.1016)
+					(bold yes)
 				)
 			)
@@
 			)
 		)
+		(property "DigiKey" ""
+			(at 0 0 0)
+			(unlocked yes)
+			(layer "F.Fab")
+			(hide yes)
+			(effects
+				(font
+					(size 1 1)
+					(thickness 0.15)
+				)
+			)
+		)
+		(property "Mouser" ""
+			(at 0 0 0)
+			(unlocked yes)
+			(layer "F.Fab")
+			(hide yes)
+			(effects
+				(font
+					(size 1 1)
+					(thickness 0.15)
+				)
+			)
+		)
+		(property "TME" ""
+			(at 0 0 0)
+			(unlocked yes)
+			(layer "F.Fab")
+			(hide yes)
+			(effects
+				(font
+					(size 1 1)
+					(thickness 0.15)
+				)
+			)
+		)
+		(property "LCSC" ""
+			(at 0 0 0)
+			(unlocked yes)
+			(layer "F.Fab")
+			(hide yes)
+			(effects
+				(font
+					(size 1 1)
+					(thickness 0.15)
+				)
+			)
+		)
 		(sheetname "/ADIB, PWM, AFE connectors/")
 		(sheetfile "ADIB_PWM.kicad_sch")
@@
 		(duplicate_pad_numbers_are_jumpers no)
 		(fp_text user "${REFERENCE}"
-			(at 0 2.5 0)
+			(at 0 0.762 0)
 			(unlocked yes)
 			(layer "F.Fab")
 			(effects
 				(font
-					(size 1 1)
-					(thickness 0.15)
+					(size 0.6096 0.6096)
+					(thickness 0.1016)
+					(bold yes)
 				)
 			)
@@
 		(pad "1" thru_hole circle
 			(at 0 0)
-			(size 1.27 1.27)
-			(drill 0.6096)
+			(size 1.8 1.8)
+			(drill 1.1)
 			(layers "*.Cu" "*.Mask")
 			(remove_unused_layers no)

Commit message: Y1 value updated
Parts:
- Y1: value LF XTAL026392 -> ABM8-16.000MHZ-10-D7G-T
Changed lines of the file:
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@@
 			)
 		)
-		(property "Value" "LF XTAL026392"
+		(property "Value" "ABM8-16.000MHZ-10-D7G-T"
 			(at 0 2.7305 0)
 			(layer "F.Fab")
@@
 			)
 		)
-		(property "DigiKey" "1923-1009-ND"
+		(property "DigiKey" "535-14383-1-ND"
 			(at 0 0 180)
 			(unlocked yes)
@@
 			)
 		)
-		(property "Mouser" "449-LFXTAL026392BULK"
+		(property "Mouser" "815-ABM816.MHZ10D7GT"
 			(at 0 0 180)
 			(unlocked yes)
@@
 			)
 		)
-		(property "TME" "16.00M-12SM"
+		(property "TME" "CX3225FB16000F0FZZ"
 			(at 0 0 180)
 			(unlocked yes)
@@
 			)
 		)
-		(property "LCSC" "C2450580"
+		(property "LCSC" "C1986769"
 			(at 0 0 180)
 			(unlocked yes)
