File: KiCad/EEZ DIB MIO168plus.kicad_pcb (KiCad board)
At the start: 4 copper layers, 191 x 95 mm, 277 parts, among them IC1 USB3300-EZK, IC10 MC78L15ACDR2G, IC11 MC79L15ACDR2G, IC12 74HC126PW,118, IC13 OPA2196IDR, IC14 DAC7760IPWPR, IC15 DAC7760IPWPR, IC16 SN74LVC138ADBR, IC17 DAC7563TDGSR, IC18 OPA376AIDBVR, IC19 PCAL9714HNMP, IC2 M24C32-DFDW6TP, IC20 OPA2196IDR, IC21 TLE75008ESDXUMA1, IC22 TL431B, IC3 ISO6762FDWR, IC4 ISO6762FDWR, IC5 ISO6762FDWR, IC6 STM32F446ZET6, IC7 IS42S16400N-6TL, IC8 SN6505BDBVT, IC9 TPS7A2033PDBVR, Q1 MMBT5401, Q10 NTJD5121NT1G, Q11 NTJD5121NT1G, Q2 MMBT5551, Q3 MMBT5551, Q4 DMP3099L, Q5 2N7002, Q6 DMP3099L, Q7 NTJD5121NT1G, Q8 NTJD5121NT1G, Q9 NTJD5121NT1G, X2 CBED202-1379B001C1AD, X4 1844824, Y1 ABM8-16.000MHZ-10-D7G-T

Commit message: BOM updated
Parts:
- ZD1, ZD2: value SMAJ16A -> SMF16A; footprint PCM_EEZ_SMD:DO214AC-2 -> PCM_EEZ_SMD:SODFL3718X130N
- ZD3: value SMAJ24A/TR13 -> SMF24A; footprint PCM_EEZ_SMD:DO214AC-2 -> PCM_EEZ_SMD:SODFL3718X130N
- moved ZD3 1.20 mm to (118.6, 130.8)
- moved D13 0.48 mm to (146.9, 137.0)
- moved D14 0.46 mm to (140.1, 137.0)
- moved ZD2 0.40 mm to (140.1, 134.9)
- moved ZD1 0.38 mm to (146.9, 134.9)
Routing:
- net ISO_PWM2: track 63.1 -> 60.2 mm
- net GND_ISO: track 137.4 -> 136.7 mm
- net PWM_OUT#1: track 76.4 -> 75.8 mm

Commit message: ZD3 modified to bidirectional TVS
Parts:
- ZD3: value SMF24A -> SMF24CA
Changed lines of the file:
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@@
 	(title_block
 		(title "${project_name}")
-		(date "2026-09-13")
+		(date "2026-09-14")
 		(rev "${project_version}")
 		(company "${project_creator}")
@@
 			)
 		)
-		(property "Value" "SMF24A"
+		(property "Value" "SMF24CA"
 			(at 0 0 0)
 			(layer "F.Fab")
@@
 			)
 		)
-		(property "DigiKey" "4878-SMF24ACT-ND"
+		(property "DigiKey" "4878-SMF24CADKR-ND"
 			(at 0 0 0)
 			(unlocked yes)
@@
 			)
 		)
-		(property "Mouser" "637-SMF24A"
+		(property "Mouser" "637-SMF24CA"
 			(at 0 0 0)
 			(unlocked yes)
@@
 			)
 		)
-		(property "TME" "SMF24A-DIO"
+		(property "TME" "SMF24CA-DIO"
 			(at 0 0 0)
 			(unlocked yes)
@@
 			)
 		)
-		(property "LCSC" "C315999"
+		(property "LCSC" "C3720035"
 			(at 0 0 0)
 			(unlocked yes)
