File: KiCad/ADIB_PWM.kicad_sch (KiCad schematic)
At the start: 65 parts, among them IC10 L78L15, IC11 L79L15, IC12 74HC126PW,118, IC8 SN6505BDBVT, IC9 TPS7A2033PDBVR, Q1 MMBT5401, Q2 MMBT5551, Q3 MMBT5551, Q4 IRLML2246TRPBF, Q5 2N7002, Q6 IRLML2246TRPBF

Commit message: Gerber files added
Parts:
- C43: LCSC (none) -> C303960
- C57: DigiKey (none) -> 490-12738-1-ND; LCSC (none) -> C77047; Mouser (none) -> 81-GRM188R61E225KA2D; TME (none) -> GRM188R61E225KA12D
- FB2, FB3: LCSC (none) -> C337877
- R11, R12: DigiKey 13-RT0805FRE07470KLDKR-ND -> A126370CT-ND; LCSC (none) -> C17709; Mouser 652-CMP0805-FX-4703L -> 71-CRCW0805470KFKEA; TME 0805S8F4703T5E -> 0805S8J0474T5E
- R16, R17: DigiKey (none) -> 311-100KHRCT-ND; LCSC (none) -> C25803; Mouser (none) -> 603-RC0603FR-07100KL; TME (none) -> SMD0603-100K-1%
- R20, R21: DigiKey (none) -> 13-RC0603FR-10100RLCT-ND; LCSC (none) -> C22775; Mouser (none) -> 603-RC0603FR-10100RL; TME (none) -> RC0603FR-10100RL
Changed lines of the file:
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@@
 			)
 		)
-		(property "DigiKey" ""
+		(property "DigiKey" "13-RC0603FR-10100RLCT-ND"
 			(at 261.62 71.12 0)
 			(hide yes)
@@
 			)
 		)
-		(property "Mouser" ""
+		(property "Mouser" "603-RC0603FR-10100RL"
 			(at 261.62 71.12 0)
 			(hide yes)
@@
 			)
 		)
-		(property "TME" ""
+		(property "TME" "RC0603FR-10100RL"
 			(at 261.62 71.12 0)
 			(hide yes)
@@
 			)
 		)
+		(property "LCSC" "C22775"
+			(at 261.62 71.12 90)
+			(hide yes)
+			(show_name no)
+			(do_not_autoplace no)
+			(effects
+				(font
+					(size 0.889 0.889)
+				)
+			)
+		)
 		(pin "1"
 		)
@@
 			)
 		)
+		(property "LCSC" "C337877"
+			(at 124.46 124.46 90)
+			(hide yes)
+			(show_name no)
+			(do_not_autoplace no)
+			(effects
+				(font
+					(size 0.889 0.889)
+				)
+			)
+		)
 		(pin "2"
 		)
@@
 			)
 		)
-		(property "DigiKey" ""
+		(property "DigiKey" "311-100KHRCT-ND"
 			(at 218.44 93.98 0)
 			(hide yes)
@@
 			)
 		)
-		(property "Mouser" ""
+		(property "Mouser" "603-RC0603FR-07100KL"
 			(at 218.44 93.98 0)
 			(hide yes)
@@
 			)
 		)
-		(property "TME" ""
+		(property "TME" "SMD0603-100K-1%"
 			(at 218.44 93.98 0)
 			(hide yes)
@@
 			)
 		)
+		(property "LCSC" "C25803"
+			(at 218.44 93.98 0)
+			(hide yes)
+			(show_name no)
+			(do_not_autoplace no)
+			(effects
+				(font
+					(size 0.889 0.889)
+				)
+			)
+		)
 		(pin "1"
 		)
@@
 			)
 		)
-		(property "DigiKey" ""
+		(property "DigiKey" "13-RC0603FR-10100RLCT-ND"
 			(at 261.62 50.8 0)
 			(hide yes)
@@
 			)
 		)
-		(property "Mouser" ""
+		(property "Mouser" "603-RC0603FR-10100RL"
 			(at 261.62 50.8 0)
 			(hide yes)
@@
 			)
 		)
-		(property "TME" ""
+		(property "TME" "RC0603FR-10100RL"
 			(at 261.62 50.8 0)
 			(hide yes)
@@
 			)
 		)
+		(property "LCSC" "C22775"
+			(at 261.62 50.8 90)
+			(hide yes)
+			(show_name no)
+			(do_not_autoplace no)
+			(effects
+				(font
+					(size 0.889 0.889)
+				)
+			)
+		)
 		(pin "1"
 		)
@@
 			)
 		)
-		(property "DigiKey" ""
+		(property "DigiKey" "311-100KHRCT-ND"
 			(at 218.44 132.08 0)
 			(hide yes)
@@
 			)
 		)
-		(property "Mouser" ""
+		(property "Mouser" "603-RC0603FR-07100KL"
 			(at 218.44 132.08 0)
 			(hide yes)
@@
 			)
 		)
-		(property "TME" ""
+		(property "TME" "SMD0603-100K-1%"
 			(at 218.44 132.08 0)
 			(hide yes)
@@
 			)
 		)
+		(property "LCSC" "C25803"
+			(at 218.44 132.08 0)
+			(hide yes)
+			(show_name no)
+			(do_not_autoplace no)
+			(effects
+				(font
+					(size 0.889 0.889)
+				)
+			)
+		)
 		(pin "1"
 		)
@@
 			)
 		)
-		(property "DigiKey" "13-RT0805FRE07470KLDKR-ND"
+		(property "DigiKey" "A126370CT-ND"
 			(at 43.18 129.54 0)
 			(hide yes)
@@
 			)
 		)
-		(property "Mouser" "652-CMP0805-FX-4703L"
+		(property "Mouser" "71-CRCW0805470KFKEA"
 			(at 43.18 129.54 0)
 			(hide yes)
@@
 			)
 		)
-		(property "TME" "0805S8F4703T5E"
+		(property "TME" "0805S8J0474T5E"
 			(at 43.18 129.54 0)
 			(hide yes)
@@
 			)
 		)
+		(property "LCSC" "C17709"
+			(at 43.18 129.54 90)
+			(hide yes)
+			(show_name no)
+			(do_not_autoplace no)
+			(effects
+				(font
+					(size 0.889 0.889)
+				)
+			)
+		)
 		(pin "1"
 		)
@@
 			)
 		)
-		(property "DigiKey" "13-RT0805FRE07470KLDKR-ND"
+		(property "DigiKey" "A126370CT-ND"
 			(at 53.34 129.54 0)
 			(hide yes)
@@
 			)
 		)
-		(property "Mouser" "652-CMP0805-FX-4703L"
+		(property "Mouser" "71-CRCW0805470KFKEA"
 			(at 53.34 129.54 0)
 			(hide yes)
@@
 			)
 		)
-		(property "TME" "0805S8F4703T5E"
+		(property "TME" "0805S8J0474T5E"
 			(at 53.34 129.54 0)
 			(hide yes)
@@
 			)
 		)
+		(property "LCSC" "C17709"
+			(at 53.34 129.54 90)
+			(hide yes)
+			(show_name no)
+			(do_not_autoplace no)
+			(effects
+				(font
+					(size 0.889 0.889)
+				)
+			)
+		)
 		(pin "1"
 		)
@@
 			)
 		)
+		(property "LCSC" "C303960"
+			(at 45.72 137.16 90)
+			(hide yes)
+			(show_name no)
+			(do_not_autoplace no)
+			(effects
+				(font
+					(size 0.889 0.889)
+				)
+			)
+		)
 		(pin "1"
 		)
@@
 			)
 		)
-		(property "DigiKey" ""
+		(property "DigiKey" "490-12738-1-ND"
 			(at 157.48 63.5 0)
 			(hide yes)
@@
 			)
 		)
-		(property "Mouser" ""
+		(property "Mouser" "81-GRM188R61E225KA2D"
 			(at 157.48 63.5 0)
 			(hide yes)
@@
 			)
 		)
-		(property "TME" ""
+		(property "TME" "GRM188R61E225KA12D"
 			(at 157.48 63.5 0)
 			(hide yes)
@@
 			)
 		)
+		(property "LCSC" "C77047"
+			(at 157.48 63.5 0)
+			(hide yes)
+			(show_name no)
+			(do_not_autoplace no)
+			(effects
+				(font
+					(size 0.889 0.889)
+				)
+			)
+		)
 		(pin "1"
 		)
@@
 				)
 			)
+		)
+		(property "LCSC" "C337877"
+			(at 124.46 83.82 90)
+			(hide yes)
+			(show_name no)
+			(do_not_autoplace no)
+			(effects
+				(font
+					(size 0.889 0.889)
+				)
+			)

Commit message: BOM update
Parts:
- D10, D11, D13, D14, D2, D3, D4, D5, D6, D7, D8, D9: LCSC (none) -> C236079
- IC10: LCSC (none) -> C233225
- IC11: LCSC (none) -> C148319
- IC12: LCSC (none) -> C507234; TME SN74HC126PW -> SN74HC126PWR
- IC8: LCSC (none) -> C2156022
- IC9: DigiKey (none) -> 296-TPS7A2033PDBVRCT-ND; LCSC (none) -> C2862740; Mouser (none) -> 595-TPS7A2033PDBVR; TME - -> TPS7A2033PDBVR
- JP2, JP3: LCSC (none) -> C3324237
- L1: LCSC (none) -> C2651160
- Q1: LCSC (none) -> C21488
- Q2, Q3: LCSC (none) -> C83942
- Q4, Q6: LCSC (none) -> C127272
- Q5: LCSC (none) -> C16338
- R13, R14: DigiKey (none) -> 13-RC0603FR-1347RLCT-ND; LCSC (none) -> C4328334; Mouser (none) -> 603-RC0603FR-1347RL; TME (none) -> SMD0603-47R-1%
- R15: DigiKey (none) -> 13-AC0603FR-7W470RLCT-ND; LCSC (none) -> C20142029; Mouser (none) -> 603-AC0603FR-7W470RL; TME (none) -> SMD0603-470R-1%
- TR1: value WE-750315371 -> 750315371; LCSC (none) -> -
- ZD1, ZD2: LCSC (none) -> C74561

Commit message: Gerbers updated
Parts:
- TP4: footprint PCM_EEZ_THT:Testhole 24_50mils -> PCM_EEZ_THT:TEST-5
Changed lines of the file:
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@@
 			)
 		)
-		(property "Footprint" "PCM_EEZ_THT:Testhole 24_50mils"
+		(property "Footprint" "PCM_EEZ_THT:TEST-5"
 			(at 170.18 106.68 0)
 			(hide yes)
@@
 				)
 			)
+		)
+		(property "DigiKey" ""
+			(at 170.18 104.14 0)
+			(hide yes)
+			(show_name no)
+			(do_not_autoplace no)
+			(effects
+				(font
+					(size 0.889 0.889)
+				)
+			)
+		)
+		(property "Mouser" ""
+			(at 170.18 104.14 0)
+			(hide yes)
+			(show_name no)
+			(do_not_autoplace no)
+			(effects
+				(font
+					(size 0.889 0.889)
+				)
+			)
+		)
+		(property "TME" ""
+			(at 170.18 104.14 0)
+			(hide yes)
+			(show_name no)
+			(do_not_autoplace no)
+			(effects
+				(font
+					(size 0.889 0.889)
+				)
+			)
+		)
+		(property "LCSC" ""
+			(at 170.18 104.14 0)
+			(hide yes)
+			(show_name no)
+			(do_not_autoplace no)
+			(effects
+				(font
+					(size 0.889 0.889)
+				)
+			)

Commit message: Updated BOM, obsolete parts have been replaced with newer ones
Parts:
- IC10: value L78L15 -> MC78L15ACDR2G
- IC11: value L79L15 -> MC79L15ACDR2G
- Q4, Q6: value IRLML2246TRPBF -> DMP3099L; DigiKey IRLML2246TRPBFTR-ND -> DMP3099L-13DICT-ND; LCSC C127272 -> C155244; Mouser 942-IRLML2246TRPBF -> 621-DMP3099L-7; TME IRLML2246TRPBF -> DMP3099L-7
Changed lines of the file:
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@@
 	(title_block
 		(title "${project_name}")
-		(date "2026-07-25")
+		(date "2026-07-27")
 		(rev "${project_version}")
 		(company "${project_creator}")
@@
 			)
 		)
-		(property "Value" "L79L15"
+		(property "Value" "MC79L15ACDR2G"
 			(at 142.24 122.555 0)
 			(show_name no)
@@
 			(effects
 				(font
-					(size 1.27 1.27)
+					(size 0.889 0.889)
 				)
 				(justify left bottom)
@@
 			)
 		)
-		(property "Value" "L78L15"
+		(property "Value" "MC78L15ACDR2G"
 			(at 139.7 85.725 0)
 			(show_name no)
@@
 			)
 		)
-		(property "Value" "IRLML2246TRPBF"
+		(property "Value" "DMP3099L"
 			(at 228.6 86.36 90)
 			(show_name no)
@@
 			)
 		)
-		(property "DigiKey" "IRLML2246TRPBFTR-ND"
+		(property "DigiKey" "DMP3099L-13DICT-ND"
 			(at 228.6 91.44 0)
 			(hide yes)
@@
 			)
 		)
-		(property "Mouser" "942-IRLML2246TRPBF "
+		(property "Mouser" "621-DMP3099L-7"
 			(at 228.6 91.44 0)
 			(hide yes)
@@
 			)
 		)
-		(property "TME" "IRLML2246TRPBF"
+		(property "TME" "DMP3099L-7"
 			(at 228.6 91.44 0)
 			(hide yes)
@@
 			)
 		)
-		(property "LCSC" "C127272"
+		(property "LCSC" "C155244"
 			(at 228.6 91.44 90)
 			(hide yes)
@@
 			)
 		)
-		(property "Value" "IRLML2246TRPBF"
+		(property "Value" "DMP3099L"
 			(at 248.92 113.665 0)
 			(show_name no)
@@
 			)
 		)
-		(property "DigiKey" "IRLML2246TRPBFTR-ND"
+		(property "DigiKey" "DMP3099L-13DICT-ND"
 			(at 243.84 111.76 0)
 			(hide yes)
@@
 			)
 		)
-		(property "Mouser" "942-IRLML2246TRPBF "
+		(property "Mouser" "621-DMP3099L-7"
 			(at 243.84 111.76 0)
 			(hide yes)
@@
 			)
 		)
-		(property "TME" "IRLML2246TRPBF"
+		(property "TME" "DMP3099L-7"
 			(at 243.84 111.76 0)
 			(hide yes)
@@
 			)
 		)
-		(property "LCSC" "C127272"
+		(property "LCSC" "C155244"
 			(at 243.84 111.76 0)
 			(hide yes)

Commit message: Image of assembled prototype
Parts:
- C46, C51, C53, C54: value 4u7 -> 4u7/35V; DigiKey 1276-1044-1-ND -> 1276-6794-1-ND; LCSC C19666 -> C913498; Mouser 187-CL10A475KP8NNNC -> 81-GRM188R6YA475ME5D; TME CL10A475KP8NNNC -> GRM219R6YA475KA73D
- C47, C48, C49, C50, C55, C56: value 1u -> 1u/50V
- TP4: Label (none) -> GND_ISO
Changed lines of the file:
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@@
 	(title_block
 		(title "${project_name}")
-		(date "2026-08-25")
+		(date "2026-08-30")
 		(rev "${project_version}")
 		(company "${project_creator}")
@@
 			)
 		)
-		(property "Value" "1u"
+		(property "Value" "1u/50V"
 			(at 93.98 116.205 90)
 			(show_name no)
@@
 			)
 		)
-		(property "Value" "4u7"
+		(property "Value" "4u7/35V"
 			(at 97.155 146.05 0)
 			(show_name no)
@@
 			)
 		)
-		(property "DigiKey" "1276-1044-1-ND"
+		(property "DigiKey" "1276-6794-1-ND"
 			(at 96.52 144.78 0)
 			(hide yes)
@@
 			)
 		)
-		(property "Mouser" "187-CL10A475KP8NNNC"
+		(property "Mouser" "81-GRM188R6YA475ME5D"
 			(at 96.52 144.78 0)
 			(hide yes)
@@
 			)
 		)
-		(property "TME" "CL10A475KP8NNNC"
+		(property "TME" "GRM219R6YA475KA73D"
 			(at 96.52 144.78 0)
 			(hide yes)
@@
 			)
 		)
-		(property "LCSC" "C19666"
+		(property "LCSC" "C913498"
 			(at 96.52 144.78 0)
 			(hide yes)
@@
 			)
 		)
+		(property "Label" "GND_ISO"
+			(at 170.18 104.14 0)
+			(hide yes)
+			(show_name no)
+			(do_not_autoplace no)
+			(effects
+				(font
+					(size 0.889 0.889)
+				)
+			)
+		)
 		(pin "1"
 		)
@@
 			)
 		)
-		(property "Value" "1u"
+		(property "Value" "1u/50V"
 			(at 132.08 113.03 0)
 			(show_name no)
@@
 			)
 		)
-		(property "Value" "1u"
+		(property "Value" "1u/50V"
 			(at 93.98 95.885 90)
 			(show_name no)
@@
 			)
 		)
-		(property "Value" "4u7"
+		(property "Value" "4u7/35V"
 			(at 96.52 66.04 0)
 			(show_name no)
@@
 			)
 		)
-		(property "DigiKey" "1276-1044-1-ND"
+		(property "DigiKey" "1276-6794-1-ND"
 			(at 96.52 66.04 0)
 			(hide yes)
@@
 			)
 		)
-		(property "Mouser" "187-CL10A475KP8NNNC"
+		(property "Mouser" "81-GRM188R6YA475ME5D"
 			(at 96.52 66.04 0)
 			(hide yes)
@@
 			)
 		)
-		(property "TME" "CL10A475KP8NNNC"
+		(property "TME" "GRM219R6YA475KA73D"
 			(at 96.52 66.04 0)
 			(hide yes)
@@
 			)
 		)
-		(property "LCSC" "C19666"
+		(property "LCSC" "C913498"
 			(at 96.52 66.04 0)
 			(hide yes)
@@
 			)
 		)
-		(property "Value" "1u"
+		(property "Value" "1u/50V"
 			(at 93.98 85.725 90)
 			(show_name no)
@@
 			)
 		)
-		(property "Value" "1u"
+		(property "Value" "1u/50V"
 			(at 132.08 97.79 0)
 			(show_name no)
@@
 			)
 		)
-		(property "Value" "1u"
+		(property "Value" "1u/50V"
 			(at 93.98 126.365 90)
 			(show_name no)
@@
 			)
 		)
-		(property "Value" "4u7"
+		(property "Value" "4u7/35V"
 			(at 116.84 97.79 0)
 			(show_name no)
@@
 			)
 		)
-		(property "DigiKey" "1276-1044-1-ND"
+		(property "DigiKey" "1276-6794-1-ND"
 			(at 116.84 93.98 0)
 			(hide yes)
@@
 			)
 		)
-		(property "Mouser" "187-CL10A475KP8NNNC"
+		(property "Mouser" "81-GRM188R6YA475ME5D"
 			(at 116.84 93.98 0)
 			(hide yes)
@@
 			)
 		)
-		(property "TME" "CL10A475KP8NNNC"
+		(property "TME" "GRM219R6YA475KA73D"
 			(at 116.84 93.98 0)
 			(hide yes)
@@
 			)
 		)
-		(property "LCSC" "C19666"
+		(property "LCSC" "C913498"
 			(at 116.84 93.98 0)
 			(hide yes)
@@
 			)
 		)
-		(property "Value" "4u7"
+		(property "Value" "4u7/35V"
 			(at 116.84 118.11 0)
 			(show_name no)
@@
 			)
 		)
-		(property "DigiKey" "1276-1044-1-ND"
+		(property "DigiKey" "1276-6794-1-ND"
 			(at 116.84 114.3 0)
 			(hide yes)
@@
 			)
 		)
-		(property "Mouser" "187-CL10A475KP8NNNC"
+		(property "Mouser" "81-GRM188R6YA475ME5D"
 			(at 116.84 114.3 0)
 			(hide yes)
@@
 			)
 		)
-		(property "TME" "CL10A475KP8NNNC"
+		(property "TME" "GRM219R6YA475KA73D"
 			(at 116.84 114.3 0)
 			(hide yes)
@@
 			)
 		)
-		(property "LCSC" "C19666"
+		(property "LCSC" "C913498"
 			(at 116.84 114.3 0)
 			(hide yes)
