File: KiCad/ADIB_PWM.kicad_sch (KiCad schematic)
At the start: 65 parts, among them IC10 MC78L15ACDR2G, IC11 MC79L15ACDR2G, IC12 74HC126PW,118, IC8 SN6505BDBVT, IC9 TPS7A2033PDBVR, Q1 MMBT5401, Q2 MMBT5551, Q3 MMBT5551, Q4 DMP3099L, Q5 2N7002, Q6 DMP3099L

Commit message: BOM updated
Parts:
- ZD1, ZD2: value SMAJ16A -> SMF16A; footprint PCM_EEZ_SMD:DO214AC-2 -> PCM_EEZ_SMD:SODFL3718X130N; DigiKey SMAJ16A-FDICT-ND -> 4878-SMF16ATR-ND; LCSC C74561 -> C207257; Mouser 621-SMAJ16A-13-F -> 637-SMF16A; TME SMAJ16A-13-F -> SMF16A-DIO
Changed lines of the file:
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@@
 			)
 		)
-		(property "Value" "SMAJ16A"
+		(property "Value" "SMF16A"
 			(at 256.032 56.896 90)
 			(show_name no)
@@
 			)
 		)
-		(property "Footprint" "PCM_EEZ_SMD:DO214AC-2"
+		(property "Footprint" "PCM_EEZ_SMD:SODFL3718X130N"
 			(at 250.825 55.245 0)
 			(hide yes)
@@
 			)
 		)
-		(property "DigiKey" "SMAJ16A-FDICT-ND"
+		(property "DigiKey" "4878-SMF16ATR-ND"
 			(at 254 55.88 0)
 			(hide yes)
@@
 			)
 		)
-		(property "Mouser" "621-SMAJ16A-13-F"
+		(property "Mouser" "637-SMF16A"
 			(at 254 55.88 0)
 			(hide yes)
@@
 			)
 		)
-		(property "TME" "SMAJ16A-13-F"
+		(property "TME" "SMF16A-DIO"
 			(at 254 55.88 0)
 			(hide yes)
@@
 			)
 		)
-		(property "LCSC" "C74561"
+		(property "LCSC" "C207257"
 			(at 254 55.88 90)
 			(hide yes)
@@
 			)
 		)
-		(property "Value" "SMAJ16A"
+		(property "Value" "SMF16A"
 			(at 261.62 84.455 90)
 			(show_name no)
@@
 			)
 		)
-		(property "Footprint" "PCM_EEZ_SMD:DO214AC-2"
+		(property "Footprint" "PCM_EEZ_SMD:SODFL3718X130N"
 			(at 255.905 84.455 0)
 			(hide yes)
@@
 			)
 		)
-		(property "DigiKey" "SMAJ16A-FDICT-ND"
+		(property "DigiKey" "4878-SMF16ATR-ND"
 			(at 259.08 83.82 0)
 			(hide yes)
@@
 			)
 		)
-		(property "Mouser" "621-SMAJ16A-13-F"
+		(property "Mouser" "637-SMF16A"
 			(at 259.08 83.82 0)
 			(hide yes)
@@
 			)
 		)
-		(property "TME" "SMAJ16A-13-F"
+		(property "TME" "SMF16A-DIO"
 			(at 259.08 83.82 0)
 			(hide yes)
@@
 			)
 		)
-		(property "LCSC" "C74561"
+		(property "LCSC" "C207257"
 			(at 259.08 83.82 90)
 			(hide yes)
