File: KiCad/Voltage_DAC_Digital_outputs.kicad_sch (KiCad schematic)
At the start: 41 parts, among them IC16 SN74LVC138ADBR, IC17 DAC7563TDGSR, IC18 OPA376AIDBVR, IC19 PCAL9714HNMP, IC20 OPA2196IDR, IC21 TLE75008ESDXUMA1

Commit message: Gerber files added
Parts:
- C90, C91: DigiKey (none) -> 1276-1018-2-ND; Mouser (none) -> 187-CL10B102KB8NNNC; TME (none) -> CL10B102KB8NNNC
- FB6: LCSC (none) -> C337877
Changed lines of the file:
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@@
 			)
 		)
-		(property "DigiKey" ""
+		(property "DigiKey" "1276-1018-2-ND"
 			(at 220.98 45.72 0)
 			(hide yes)
@@
 			)
 		)
-		(property "Mouser" ""
+		(property "Mouser" "187-CL10B102KB8NNNC "
 			(at 220.98 45.72 0)
 			(hide yes)
@@
 			)
 		)
-		(property "TME" ""
+		(property "TME" "CL10B102KB8NNNC"
 			(at 220.98 45.72 0)
 			(hide yes)
@@
 			)
 		)
-		(property "DigiKey" ""
+		(property "DigiKey" "1276-1018-2-ND"
 			(at 220.98 81.28 0)
 			(hide yes)
@@
 			)
 		)
-		(property "Mouser" ""
+		(property "Mouser" "187-CL10B102KB8NNNC "
 			(at 220.98 81.28 0)
 			(hide yes)
@@
 			)
 		)
-		(property "TME" ""
+		(property "TME" "CL10B102KB8NNNC"
 			(at 220.98 81.28 0)
 			(hide yes)
@@
 				)
 			)
+		)
+		(property "LCSC" "C337877"
+			(at 109.22 66.04 90)
+			(hide yes)
+			(show_name no)
+			(do_not_autoplace no)
+			(effects
+				(font
+					(size 0.889 0.889)
+				)
+			)

Commit message: BOM update
Parts:
- C90, C91: LCSC (none) -> C1588
- IC17: LCSC (none) -> C2879196
- IC18: LCSC (none) -> C42134
- IC20: DigiKey 296-1282-1-ND -> 296-48159-1-ND; LCSC (none) -> C2057972; Mouser 595-TL072CDR -> 595-OPA2196IDR; TME TL072CD-ST -> OPA2196IDR
- IC21: LCSC (none) -> C2150432
- R29, R30, R31, R32, R33, R34: DigiKey (none) -> 13-RC0603BR-079K09LCT-ND; LCSC (none) -> C185301; Mouser (none) -> 603-RC0603BR-079K09L; TME (none) -> AR0603-9K09-0.1%
- R35, R36, R37, R39: DigiKey (none) -> YAG1730CT-ND; LCSC (none) -> C723587; Mouser (none) -> 603-RT0603BRD0775KL; TME (none) -> AR0603-75K-0.1%
- R38, R40: DigiKey (none) -> 13-RC0603FR-13180RLCT-ND; LCSC (none) -> C4077604; Mouser (none) -> 603-RC0603FR-13180RL; TME (none) -> SMD0603-180R-1%
- R41, R42: DigiKey (none) -> 13-RC0603FR-1347RLCT-ND; LCSC (none) -> C4328334; Mouser (none) -> 603-RC0603FR-1347RL; TME (none) -> SMD0603-47R-1%
- TVS3, TVS4: LCSC (none) -> C38558

Commit message: Updated BOM, obsolete parts have been replaced with newer ones
Parts:
- TVS3, TVS4: value PESD12VL1BA,115 -> PESD12VL1BA; DigiKey 1727-3808-1-ND -> 4518-PESD12VL1BACT-ND; Mouser 771-PESD12VL1BA-T/R -> 771-PESD12VS1UAF; TME PESD12VL1BA.115 -> PESD12VL1BA,115
Connections:
- net ~{ISO_RESET}: no longer IC21.21 (IDLE)
- no-connect marks 0 -> 1
Changed lines of the file:
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@@
 		(color 0 0 0 0)
 	)
+	(no_connect
+		(at 215.9 134.62)
+	)
 	(wire
 		(pts
@@
 	(wire
 		(pts
-			(xy 208.28 134.62) (xy 215.9 134.62)
-		)
-		(stroke
-			(width 0)
-			(type default)
-		)
-	)
-	(wire
-		(pts
 			(xy 259.08 63.5) (xy 259.08 66.04)
 		)
@@
 	(global_label "~{ISO_RESET}"
 		(shape input)
-		(at 208.28 134.62 180)
-		(fields_autoplaced yes)
-		(effects
-			(font
-				(size 0.889 0.889)
-			)
-			(justify right)
-		)
-		(property "Intersheetrefs" "${INTERSHEET_REFS}"
-			(at 199.2903 134.62 0)
-			(hide yes)
-			(show_name no)
-			(do_not_autoplace no)
-			(effects
-				(font
-					(size 1.27 1.27)
-				)
-				(justify right)
-			)
-		)
-	)
-	(global_label "~{ISO_RESET}"
-		(shape input)
 		(at 38.1 66.04 180)
 		(fields_autoplaced yes)
@@
 			)
 		)
-		(property "Value" "PESD12VL1BA,115"
+		(property "Value" "PESD12VL1BA"
 			(at 202.692 48.641 90)
 			(show_name no)
@@
 			)
 		)
-		(property "DigiKey" "1727-3808-1-ND"
+		(property "DigiKey" "4518-PESD12VL1BACT-ND"
 			(at 195.58 43.18 0)
 			(hide yes)
@@
 			)
 		)
-		(property "Mouser" "771-PESD12VL1BA-T/R"
+		(property "Mouser" "771-PESD12VS1UAF"
 			(at 193.04 43.18 0)
 			(hide yes)
@@
 			)
 		)
-		(property "TME" "PESD12VL1BA.115"
+		(property "TME" "PESD12VL1BA,115"
 			(at 190.5 43.18 0)
 			(hide yes)
@@
 			)
 		)
-		(property "Value" "PESD12VL1BA,115"
+		(property "Value" "PESD12VL1BA"
 			(at 202.692 84.201 90)
 			(show_name no)
@@
 			)
 		)
-		(property "DigiKey" "1727-3808-1-ND"
+		(property "DigiKey" "4518-PESD12VL1BACT-ND"
 			(at 195.58 78.74 0)
 			(hide yes)
@@
 			)
 		)
-		(property "Mouser" "771-PESD12VL1BA-T/R"
+		(property "Mouser" "771-PESD12VS1UAF"
 			(at 193.04 78.74 0)
 			(hide yes)
@@
 			)
 		)
-		(property "TME" "PESD12VL1BA.115"
+		(property "TME" "PESD12VL1BA,115"
 			(at 190.5 78.74 0)
 			(hide yes)

Commit message: OSHWA ID added
Parts:
- R29, R30, R31, R32, R33, R34: DigiKey 13-RC0603BR-079K09LCT-ND -> YAG4788CT-ND
Changed lines of the file:
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@@
 	(title_block
 		(title "${project_name}")
-		(date "2026-07-25")
+		(date "2026-08-07")
 		(rev "${project_version}")
 		(company "${project_creator}")
@@
 			)
 		)
-		(property "DigiKey" "13-RC0603BR-079K09LCT-ND"
+		(property "DigiKey" "YAG4788CT-ND"
 			(at 154.94 63.5 0)
 			(hide yes)
@@
 			)
 		)
-		(property "DigiKey" "13-RC0603BR-079K09LCT-ND"
+		(property "DigiKey" "YAG4788CT-ND"
 			(at 99.06 38.1 0)
 			(hide yes)
@@
 			)
 		)
-		(property "DigiKey" "13-RC0603BR-079K09LCT-ND"
+		(property "DigiKey" "YAG4788CT-ND"
 			(at 154.94 27.94 0)
 			(hide yes)
@@
 			)
 		)
-		(property "DigiKey" "13-RC0603BR-079K09LCT-ND"
+		(property "DigiKey" "YAG4788CT-ND"
 			(at 99.06 48.26 0)
 			(hide yes)
@@
 			)
 		)
-		(property "DigiKey" "13-RC0603BR-079K09LCT-ND"
+		(property "DigiKey" "YAG4788CT-ND"
 			(at 154.94 43.18 0)
 			(hide yes)
@@
 			)
 		)
-		(property "DigiKey" "13-RC0603BR-079K09LCT-ND"
+		(property "DigiKey" "YAG4788CT-ND"
 			(at 154.94 78.74 0)
 			(hide yes)

Commit message: BOM update
Parts:
- D16: now not fitted; now left out of the parts list
- TVS3, TVS4: value PESD12VL1BA -> SD12C-7; DigiKey 4518-PESD12VL1BACT-ND -> 31-SD12C-7CT-ND; LCSC C38558 -> C1977377; Mouser 771-PESD12VS1UAF -> 621-SD12C-7; TME PESD12VL1BA,115 -> SD12C-7
Changed lines of the file:
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@@
 	(title_block
 		(title "${project_name}")
-		(date "2026-08-07")
+		(date "2026-08-23")
 		(rev "${project_version}")
 		(company "${project_creator}")
@@
 			)
 		)
-		(property "Value" "PESD12VL1BA"
+		(property "Value" "SD12C-7"
 			(at 202.692 48.641 90)
 			(show_name no)
@@
 			)
 		)
-		(property "DigiKey" "4518-PESD12VL1BACT-ND"
+		(property "DigiKey" "31-SD12C-7CT-ND"
 			(at 195.58 43.18 0)
 			(hide yes)
@@
 			)
 		)
-		(property "Mouser" "771-PESD12VS1UAF"
+		(property "Mouser" "621-SD12C-7"
 			(at 193.04 43.18 0)
 			(hide yes)
@@
 			)
 		)
-		(property "TME" "PESD12VL1BA,115"
+		(property "TME" "SD12C-7"
 			(at 190.5 43.18 0)
 			(hide yes)
@@
 			)
 		)
-		(property "LCSC" "C38558"
+		(property "LCSC" "C1977377"
 			(at 200.66 43.18 90)
 			(hide yes)
@@
 			)
 		)
-		(property "Value" "PESD12VL1BA"
+		(property "Value" "SD12C-7"
 			(at 202.692 84.201 90)
 			(show_name no)
@@
 			)
 		)
-		(property "DigiKey" "4518-PESD12VL1BACT-ND"
+		(property "DigiKey" "31-SD12C-7CT-ND"
 			(at 195.58 78.74 0)
 			(hide yes)
@@
 			)
 		)
-		(property "Mouser" "771-PESD12VS1UAF"
+		(property "Mouser" "621-SD12C-7"
 			(at 193.04 78.74 0)
 			(hide yes)
@@
 			)
 		)
-		(property "TME" "PESD12VL1BA,115"
+		(property "TME" "SD12C-7"
 			(at 190.5 78.74 0)
 			(hide yes)
@@
 			)
 		)
-		(property "LCSC" "C38558"
+		(property "LCSC" "C1977377"
 			(at 200.66 78.74 90)
 			(hide yes)
@@
 		(body_style 1)
 		(exclude_from_sim no)
-		(in_bom yes)
+		(in_bom no)
 		(on_board yes)
 		(in_pos_files yes)
-		(dnp no)
+		(dnp yes)
 		(fields_autoplaced yes)
 		(property "Reference" "D16"
@@
 		(body_style 1)
 		(exclude_from_sim no)
-		(in_bom yes)
+		(in_bom no)
 		(on_board yes)
 		(in_pos_files yes)
-		(dnp no)
+		(dnp yes)
 		(fields_autoplaced yes)
 		(property "Reference" "D16"

Commit message: X2 connector position adjustment
Connections:
- net +3V3_ISO: now also IC21.21 (IDLE)
- no-connect marks 1 -> 0
Changed lines of the file:
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@@
 	(title_block
 		(title "${project_name}")
-		(date "2026-08-23")
+		(date "2026-08-25")
 		(rev "${project_version}")
 		(company "${project_creator}")
@@
 	)
 	(junction
+		(at 213.36 119.38)
+		(diameter 0)
+		(color 0 0 0 0)
+	)
+	(junction
 		(at 119.38 149.86)
 		(diameter 0)
@@
 		(diameter 0)
 		(color 0 0 0 0)
-	)
-	(no_connect
-		(at 215.9 134.62)
 	)
 	(wire
@@
 	(wire
 		(pts
+			(xy 213.36 134.62) (xy 215.9 134.62)
+		)
+		(stroke
+			(width 0)
+			(type default)
+		)
+	)
+	(wire
+		(pts
 			(xy 165.1 38.1) (xy 165.1 33.02)
 		)
@@
 		)
 		(stroke
+			(width 0)
+			(type default)
+		)
+	)
+	(wire
+		(pts
+			(xy 213.36 119.38) (xy 213.36 134.62)
+		)
+		(stroke

Commit message: Image of assembled prototype
Parts:
- C84: value 4u7 -> 4u7/35V; DigiKey 1276-1044-1-ND -> 1276-6794-1-ND; LCSC C19666 -> C913498; Mouser 187-CL10A475KP8NNNC -> 81-GRM188R6YA475ME5D; TME CL10A475KP8NNNC -> GRM219R6YA475KA73D
Changed lines of the file:
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@@
 	(title_block
 		(title "${project_name}")
-		(date "2026-08-25")
+		(date "2026-08-30")
 		(rev "${project_version}")
 		(company "${project_creator}")
@@
 			)
 		)
-		(property "Value" "4u7"
+		(property "Value" "4u7/35V"
 			(at 91.44 74.93 0)
 			(show_name no)
@@
 			)
 		)
-		(property "DigiKey" "1276-1044-1-ND"
+		(property "DigiKey" "1276-6794-1-ND"
 			(at 91.44 73.66 0)
 			(hide yes)
@@
 			)
 		)
-		(property "Mouser" "187-CL10A475KP8NNNC"
+		(property "Mouser" "81-GRM188R6YA475ME5D"
 			(at 91.44 73.66 0)
 			(hide yes)
@@
 			)
 		)
-		(property "TME" "CL10A475KP8NNNC"
+		(property "TME" "GRM219R6YA475KA73D"
 			(at 91.44 73.66 0)
 			(hide yes)
@@
 			)
 		)
-		(property "LCSC" "C19666"
+		(property "LCSC" "C913498"
 			(at 91.44 73.66 0)
 			(hide yes)

Commit message: BOM updated
Parts:
- ZD3: value SMAJ24A/TR13 -> SMF24A; footprint PCM_EEZ_SMD:DO214AC-2 -> PCM_EEZ_SMD:SODFL3718X130N; DigiKey 13-SMAJ24A/TR13CT-ND -> 4878-SMF24ACT-ND; LCSC C90510 -> C315999; Mouser 603-SMAJ24A/TR13 -> 637-SMF24A; TME SMAJ24A-LF -> SMF24A-DIO
Changed lines of the file:
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@@
 			)
 		)
-		(property "Value" "SMAJ24A/TR13"
+		(property "Value" "SMF24A"
 			(at 256.032 112.776 90)
 			(show_name no)
@@
 			)
 		)
-		(property "Footprint" "PCM_EEZ_SMD:DO214AC-2"
+		(property "Footprint" "PCM_EEZ_SMD:SODFL3718X130N"
 			(at 250.825 111.125 0)
 			(hide yes)
@@
 			)
 		)
-		(property "DigiKey" "13-SMAJ24A/TR13CT-ND"
+		(property "DigiKey" "4878-SMF24ACT-ND"
 			(at 254 111.76 0)
 			(hide yes)
@@
 			)
 		)
-		(property "Mouser" "603-SMAJ24A/TR13"
+		(property "Mouser" "637-SMF24A"
 			(at 254 111.76 0)
 			(hide yes)
@@
 			)
 		)
-		(property "TME" "SMAJ24A-LF"
+		(property "TME" "SMF24A-DIO"
 			(at 254 111.76 0)
 			(hide yes)
@@
 			)
 		)
-		(property "LCSC" "C90510"
+		(property "LCSC" "C315999"
 			(at 254 111.76 0)
 			(hide yes)
