File: KiCad/Voltage_DAC_Digital_outputs.kicad_sch (KiCad schematic)
At the start: 41 parts, among them IC16 SN74LVC138ADBR, IC17 DAC7563TDGSR, IC18 OPA376AIDBVR, IC19 PCAL9714HNMP, IC20 OPA2196IDR, IC21 TLE75008ESDXUMA1

Commit message: ZD3 modified to bidirectional TVS
Parts:
- ZD3: value SMF24A -> SMF24CA; symbol PCM_EEZ_discretes:DIODE_TVS_UNI -> PCM_EEZ_discretes:DIODE_TVS; DigiKey 4878-SMF24ACT-ND -> 4878-SMF24CADKR-ND; LCSC C315999 -> C3720035; Mouser 637-SMF24A -> 637-SMF24CA; TME SMF24A-DIO -> SMF24CA-DIO
Changed lines of the file:
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@@
 	(title_block
 		(title "${project_name}")
-		(date "2026-08-30")
+		(date "2026-09-14")
 		(rev "${project_version}")
 		(company "${project_creator}")
@@
 	)
 	(symbol
-		(lib_id "PCM_EEZ_discretes:DIODE_TVS_UNI")
+		(lib_id "PCM_EEZ_discretes:DIODE_TVS")
 		(at 254 111.76 270)
 		(unit 1)
@@
 		(dnp no)
 		(property "Reference" "ZD3"
-			(at 256.032 110.49 90)
+			(at 256.54 113.665 90)
 			(show_name no)
 			(do_not_autoplace no)
@@
 					(size 1.27 1.27)
 				)
-				(justify left top)
+				(justify left bottom)
 			)
 		)
-		(property "Value" "SMF24A"
-			(at 256.032 112.776 90)
+		(property "Value" "SMF24CA"
+			(at 256.54 115.57 90)
 			(show_name no)
 			(do_not_autoplace no)
@@
 					(size 1.27 1.27)
 				)
-				(justify left top)
+				(justify left bottom)
 			)
 		)
@@
 			)
 		)
-		(property "DigiKey" "4878-SMF24ACT-ND"
+		(property "DigiKey" "4878-SMF24CADKR-ND"
 			(at 254 111.76 0)
 			(hide yes)
@@
 			)
 		)
-		(property "Mouser" "637-SMF24A"
+		(property "Mouser" "637-SMF24CA"
 			(at 254 111.76 0)
 			(hide yes)
@@
 			)
 		)
-		(property "TME" "SMF24A-DIO"
+		(property "TME" "SMF24CA-DIO"
 			(at 254 111.76 0)
 			(hide yes)
@@
 			)
 		)
-		(property "LCSC" "C315999"
+		(property "LCSC" "C3720035"
 			(at 254 111.76 0)
 			(hide yes)

Commit message: #4
Parts:
- renumbered C81 to C66, C82 to C67, C83 to C68, C84 to C69, C85 to C70, C86 to C71, C87 to C72, C88 to C73, C89 to C74, C90 to C75, C91 to C76, C92 to C77, C93 to C78, C94 to C79, R29 to R30, R30 to R31, R31 to R32, R32 to R33, R33 to R34, R34 to R35, R35 to R36, R36 to R37, R37 to R38, R38 to R39, R39 to R40, R40 to R41, R41 to R42, R42 to R43, TP7 to TP8, TP8 to TP9
