File: KiCad/Digital_inputs.kicad_sch (KiCad schematic)
At the start: 49 parts, among them IC22 TL431B, Q10 2N7002PS,115, Q11 2N7002PS,115, Q7 2N7002PS,115, Q8 2N7002PS,115, Q9 2N7002PS,115

Commit message: Gerber files added
Parts:
- R52, R54, R56, R58, R60, R62, R64, R66: DigiKey (none) -> 13-RC0603FR-131KLCT-ND; LCSC (none) -> C21190; Mouser (none) -> 603-RC0603FR-131KL; TME (none) -> CQ0603-1K-1%
- R67: DigiKey (none) -> 13-RC0603FR-10100RLCT-ND; LCSC (none) -> C22775; Mouser (none) -> 603-RC0603FR-10100RL; TME (none) -> RC0603FR-10100RL
- R69: DigiKey (none) -> 13-RC0603FR-131K8LCT-ND; LCSC (none) -> C4177; Mouser (none) -> 603-RC0603FR-131K8L; TME (none) -> SMD0603-1K8-1%
Changed lines of the file:
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@@
 			)
 		)
-		(property "DigiKey" ""
+		(property "DigiKey" "13-RC0603FR-131KLCT-ND"
 			(at 157.48 132.08 0)
 			(hide yes)
@@
 			)
 		)
-		(property "Mouser" ""
+		(property "Mouser" "603-RC0603FR-131KL"
 			(at 157.48 132.08 0)
 			(hide yes)
@@
 			)
 		)
-		(property "TME" ""
+		(property "TME" "CQ0603-1K-1%"
 			(at 157.48 132.08 0)
 			(hide yes)
@@
 			)
 		)
+		(property "LCSC" "C21190"
+			(at 157.48 132.08 0)
+			(hide yes)
+			(show_name no)
+			(do_not_autoplace no)
+			(effects
+				(font
+					(size 0.889 0.889)
+				)
+			)
+		)
 		(pin "1"
 		)
@@
 			)
 		)
-		(property "DigiKey" ""
+		(property "DigiKey" "13-RC0603FR-131KLCT-ND"
 			(at 104.14 132.08 0)
 			(hide yes)
@@
 			)
 		)
-		(property "Mouser" ""
+		(property "Mouser" "603-RC0603FR-131KL"
 			(at 104.14 132.08 0)
 			(hide yes)
@@
 			)
 		)
-		(property "TME" ""
+		(property "TME" "CQ0603-1K-1%"
 			(at 104.14 132.08 0)
 			(hide yes)
@@
 			)
 		)
+		(property "LCSC" "C21190"
+			(at 104.14 132.08 0)
+			(hide yes)
+			(show_name no)
+			(do_not_autoplace no)
+			(effects
+				(font
+					(size 0.889 0.889)
+				)
+			)
+		)
 		(pin "1"
 		)
@@
 			)
 		)
-		(property "DigiKey" ""
+		(property "DigiKey" "13-RC0603FR-131KLCT-ND"
 			(at 121.92 132.08 0)
 			(hide yes)
@@
 			)
 		)
-		(property "Mouser" ""
+		(property "Mouser" "603-RC0603FR-131KL"
 			(at 121.92 132.08 0)
 			(hide yes)
@@
 			)
 		)
-		(property "TME" ""
+		(property "TME" "CQ0603-1K-1%"
 			(at 121.92 132.08 0)
 			(hide yes)
@@
 			)
 		)
-		(property "LCSC" ""
+		(property "LCSC" "C21190"
 			(at 121.92 132.08 0)
 			(hide yes)
@@
 			)
 		)
-		(property "DigiKey" ""
+		(property "DigiKey" "13-RC0603FR-131KLCT-ND"
 			(at 86.36 132.08 0)
 			(hide yes)
@@
 			)
 		)
-		(property "Mouser" ""
+		(property "Mouser" "603-RC0603FR-131KL"
 			(at 86.36 132.08 0)
 			(hide yes)
@@
 			)
 		)
-		(property "TME" ""
+		(property "TME" "CQ0603-1K-1%"
 			(at 86.36 132.08 0)
 			(hide yes)
@@
 			)
 		)
+		(property "LCSC" "C21190"
+			(at 86.36 132.08 0)
+			(hide yes)
+			(show_name no)
+			(do_not_autoplace no)
+			(effects
+				(font
+					(size 0.889 0.889)
+				)
+			)
+		)
 		(pin "1"
 		)
@@
 			)
 		)
-		(property "DigiKey" ""
+		(property "DigiKey" "13-RC0603FR-10100RLCT-ND"
 			(at 226.06 25.4 0)
 			(hide yes)
@@
 			)
 		)
-		(property "Mouser" ""
+		(property "Mouser" "603-RC0603FR-10100RL"
 			(at 226.06 25.4 0)
 			(hide yes)
@@
 			)
 		)
-		(property "TME" ""
+		(property "TME" "RC0603FR-10100RL"
 			(at 226.06 25.4 0)
 			(hide yes)
@@
 			)
 		)
-		(property "LCSC" ""
+		(property "LCSC" "C22775"
 			(at 226.06 25.4 0)
 			(hide yes)
@@
 			)
 		)
-		(property "DigiKey" ""
+		(property "DigiKey" "13-RC0603FR-131KLCT-ND"
 			(at 175.26 132.08 0)
 			(hide yes)
@@
 			)
 		)
-		(property "Mouser" ""
+		(property "Mouser" "603-RC0603FR-131KL"
 			(at 175.26 132.08 0)
 			(hide yes)
@@
 			)
 		)
-		(property "TME" ""
+		(property "TME" "CQ0603-1K-1%"
 			(at 175.26 132.08 0)
 			(hide yes)
@@
 			)
 		)
+		(property "LCSC" "C21190"
+			(at 175.26 132.08 0)
+			(hide yes)
+			(show_name no)
+			(do_not_autoplace no)
+			(effects
+				(font
+					(size 0.889 0.889)
+				)
+			)
+		)
 		(pin "2"
 		)
@@
 			)
 		)
-		(property "DigiKey" ""
+		(property "DigiKey" "13-RC0603FR-131KLCT-ND"
 			(at 139.7 132.08 0)
 			(hide yes)
@@
 			)
 		)
-		(property "Mouser" ""
+		(property "Mouser" "603-RC0603FR-131KL"
 			(at 139.7 132.08 0)
 			(hide yes)
@@
 			)
 		)
-		(property "TME" ""
+		(property "TME" "CQ0603-1K-1%"
 			(at 139.7 132.08 0)
 			(hide yes)
@@
 			)
 		)
-		(property "LCSC" ""
+		(property "LCSC" "C21190"
 			(at 139.7 132.08 0)
 			(hide yes)
@@
 			)
 		)
-		(property "DigiKey" ""
+		(property "DigiKey" "13-RC0603FR-131K8LCT-ND"
 			(at 241.3 40.64 0)
 			(hide yes)
@@
 			)
 		)
-		(property "Mouser" ""
+		(property "Mouser" "603-RC0603FR-131K8L"
 			(at 241.3 40.64 0)
 			(hide yes)
@@
 			)
 		)
-		(property "TME" ""
+		(property "TME" "SMD0603-1K8-1%"
 			(at 241.3 40.64 0)
 			(hide yes)
@@
 			)
 		)
-		(property "LCSC" ""
+		(property "LCSC" "C4177"
 			(at 241.3 40.64 0)
 			(hide yes)
@@
 			)
 		)
-		(property "DigiKey" ""
+		(property "DigiKey" "13-RC0603FR-131KLCT-ND"
 			(at 68.58 132.08 0)
 			(hide yes)
@@
 			)
 		)
-		(property "Mouser" ""
+		(property "Mouser" "603-RC0603FR-131KL"
 			(at 68.58 132.08 0)
 			(hide yes)
@@
 			)
 		)
-		(property "TME" ""
+		(property "TME" "CQ0603-1K-1%"
 			(at 68.58 132.08 0)
 			(hide yes)
@@
 			)
 		)
+		(property "LCSC" "C21190"
+			(at 68.58 132.08 0)
+			(hide yes)
+			(show_name no)
+			(do_not_autoplace no)
+			(effects
+				(font
+					(size 0.889 0.889)
+				)
+			)
+		)
 		(pin "1"
 		)
@@
 			)
 		)
-		(property "DigiKey" ""
+		(property "DigiKey" "13-RC0603FR-131KLCT-ND"
 			(at 193.04 132.08 0)
 			(hide yes)
@@
 			)
 		)
-		(property "Mouser" ""
+		(property "Mouser" "603-RC0603FR-131KL"
 			(at 193.04 132.08 0)
 			(hide yes)
@@
 			)
 		)
-		(property "TME" ""
+		(property "TME" "CQ0603-1K-1%"
 			(at 193.04 132.08 0)
 			(hide yes)
@@
 				)
 			)
+		)
+		(property "LCSC" "C21190"
+			(at 193.04 132.08 0)
+			(hide yes)
+			(show_name no)
+			(do_not_autoplace no)
+			(effects
+				(font
+					(size 0.889 0.889)
+				)
+			)

Commit message: BOM update
Parts:
- C106, C95, C99: DigiKey (none) -> 490-11153-1-ND; LCSC (none) -> C3868042; Mouser (none) -> 81-GCM1885C1H101JA6J; TME (none) -> GCM1885C1H101JA16J
- IC22: LCSC (none) -> C21235
- Q10, Q11, Q7, Q8, Q9: LCSC (none) -> C551419
- R43, R44, R45, R46, R47, R48, R49, R50: LCSC (none) -> C205261
- R51, R53, R55, R57, R59, R61, R63, R65: DigiKey (none) -> 311-27.0KHRCT-ND; LCSC (none) -> C114614; Mouser (none) -> 603-RC0603FR-0727KL; TME (none) -> SMD0603-27K-1%
- R68: DigiKey (none) -> 13-AC0603FR-7W470RLCT-ND; LCSC (none) -> C20142029; Mouser (none) -> 603-AC0603FR-7W470RL; TME (none) -> SMD0603-470R-1%

Commit message: Updated BOM, obsolete parts have been replaced with newer ones
Parts:
- Q10, Q11, Q7, Q8, Q9: value 2N7002PS,115 -> NTJD5121NT1G; DigiKey 1727-4791-2-ND -> NTJD5121NT1GOSCT-ND; LCSC C551419 -> C15215; Mouser 771-2N7002PS-115 -> 863-NTJD5121NT1G; TME 2N7002PS.115 -> NTJD5121NT1G
Changed lines of the file:
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@@
 			)
 		)
-		(property "Value" "2N7002PS,115"
+		(property "Value" "NTJD5121NT1G"
 			(at 140.335 146.05 0)
 			(show_name no)
@@
 			)
 		)
-		(property "DigiKey" "1727-4791-2-ND"
+		(property "DigiKey" "NTJD5121NT1GOSCT-ND"
 			(at 142.24 152.4 0)
 			(hide yes)
@@
 			)
 		)
-		(property "Mouser" "771-2N7002PS-115"
+		(property "Mouser" "863-NTJD5121NT1G"
 			(at 142.24 154.94 0)
 			(hide yes)
@@
 			)
 		)
-		(property "TME" "2N7002PS.115"
+		(property "TME" "NTJD5121NT1G"
 			(at 142.24 157.48 0)
 			(hide yes)
@@
 			)
 		)
-		(property "LCSC" "C551419"
+		(property "LCSC" "C15215"
 			(at 142.24 142.24 0)
 			(hide yes)
@@
 			)
 		)
-		(property "Value" "2N7002PS,115"
+		(property "Value" "NTJD5121NT1G"
 			(at 206.375 143.51 0)
 			(show_name no)
@@
 			)
 		)
-		(property "DigiKey" "1727-4791-2-ND"
+		(property "DigiKey" "NTJD5121NT1GOSCT-ND"
 			(at 208.28 149.86 0)
 			(hide yes)
@@
 			)
 		)
-		(property "Mouser" "771-2N7002PS-115"
+		(property "Mouser" "863-NTJD5121NT1G"
 			(at 208.28 152.4 0)
 			(hide yes)
@@
 			)
 		)
-		(property "TME" "2N7002PS.115"
+		(property "TME" "NTJD5121NT1G"
 			(at 208.28 154.94 0)
 			(hide yes)
@@
 			)
 		)
-		(property "LCSC" "C551419"
+		(property "LCSC" "C15215"
 			(at 208.28 139.7 0)
 			(hide yes)
@@
 			)
 		)
-		(property "Value" "2N7002PS,115"
+		(property "Value" "NTJD5121NT1G"
 			(at 219.71 139.7 0)
 			(hide yes)
@@
 			)
 		)
-		(property "DigiKey" "1727-4791-2-ND"
+		(property "DigiKey" "NTJD5121NT1GOSCT-ND"
 			(at 226.06 149.86 0)
 			(hide yes)
@@
 			)
 		)
-		(property "Mouser" "771-2N7002PS-115"
+		(property "Mouser" "863-NTJD5121NT1G"
 			(at 226.06 152.4 0)
 			(hide yes)
@@
 			)
 		)
-		(property "TME" "2N7002PS.115"
+		(property "TME" "NTJD5121NT1G"
 			(at 226.06 154.94 0)
 			(hide yes)
@@
 			)
 		)
-		(property "LCSC" "C551419"
+		(property "LCSC" "C15215"
 			(at 226.06 139.7 0)
 			(hide yes)
@@
 			)
 		)
-		(property "Value" "2N7002PS,115"
+		(property "Value" "NTJD5121NT1G"
 			(at 175.895 146.05 0)
 			(show_name no)
@@
 			)
 		)
-		(property "DigiKey" "1727-4791-2-ND"
+		(property "DigiKey" "NTJD5121NT1GOSCT-ND"
 			(at 177.8 152.4 0)
 			(hide yes)
@@
 			)
 		)
-		(property "Mouser" "771-2N7002PS-115"
+		(property "Mouser" "863-NTJD5121NT1G"
 			(at 177.8 154.94 0)
 			(hide yes)
@@
 			)
 		)
-		(property "TME" "2N7002PS.115"
+		(property "TME" "NTJD5121NT1G"
 			(at 177.8 157.48 0)
 			(hide yes)
@@
 			)
 		)
-		(property "LCSC" "C551419"
+		(property "LCSC" "C15215"
 			(at 177.8 142.24 0)
 			(hide yes)
@@
 			)
 		)
-		(property "Value" "2N7002PS,115"
+		(property "Value" "NTJD5121NT1G"
 			(at 189.23 142.24 0)
 			(hide yes)
@@
 			)
 		)
-		(property "DigiKey" "1727-4791-2-ND"
+		(property "DigiKey" "NTJD5121NT1GOSCT-ND"
 			(at 195.58 152.4 0)
 			(hide yes)
@@
 			)
 		)
-		(property "Mouser" "771-2N7002PS-115"
+		(property "Mouser" "863-NTJD5121NT1G"
 			(at 195.58 154.94 0)
 			(hide yes)
@@
 			)
 		)
-		(property "TME" "2N7002PS.115"
+		(property "TME" "NTJD5121NT1G"
 			(at 195.58 157.48 0)
 			(hide yes)
@@
 			)
 		)
-		(property "LCSC" "C551419"
+		(property "LCSC" "C15215"
 			(at 195.58 142.24 0)
 			(hide yes)
@@
 			)
 		)
-		(property "Value" "2N7002PS,115"
+		(property "Value" "NTJD5121NT1G"
 			(at 82.55 142.24 0)
 			(hide yes)
@@
 			)
 		)
-		(property "DigiKey" "1727-4791-2-ND"
+		(property "DigiKey" "NTJD5121NT1GOSCT-ND"
 			(at 88.9 152.4 0)
 			(hide yes)
@@
 			)
 		)
-		(property "Mouser" "771-2N7002PS-115"
+		(property "Mouser" "863-NTJD5121NT1G"
 			(at 88.9 154.94 0)
 			(hide yes)
@@
 			)
 		)
-		(property "TME" "2N7002PS.115"
+		(property "TME" "NTJD5121NT1G"
 			(at 88.9 157.48 0)
 			(hide yes)
@@
 			)
 		)
-		(property "LCSC" "C551419"
+		(property "LCSC" "C15215"
 			(at 88.9 142.24 0)
 			(hide yes)
@@
 			)
 		)
-		(property "Value" "2N7002PS,115"
+		(property "Value" "NTJD5121NT1G"
 			(at 104.775 146.05 0)
 			(show_name no)
@@
 			)
 		)
-		(property "DigiKey" "1727-4791-2-ND"
+		(property "DigiKey" "NTJD5121NT1GOSCT-ND"
 			(at 106.68 152.4 0)
 			(hide yes)
@@
 			)
 		)
-		(property "Mouser" "771-2N7002PS-115"
+		(property "Mouser" "863-NTJD5121NT1G"
 			(at 106.68 154.94 0)
 			(hide yes)
@@
 			)
 		)
-		(property "TME" "2N7002PS.115"
+		(property "TME" "NTJD5121NT1G"
 			(at 106.68 157.48 0)
 			(hide yes)
@@
 			)
 		)
-		(property "LCSC" "C551419"
+		(property "LCSC" "C15215"
 			(at 106.68 142.24 0)
 			(hide yes)
@@
 			)
 		)
-		(property "Value" "2N7002PS,115"
+		(property "Value" "NTJD5121NT1G"
 			(at 118.11 142.24 0)
 			(hide yes)
@@
 			)
 		)
-		(property "DigiKey" "1727-4791-2-ND"
+		(property "DigiKey" "NTJD5121NT1GOSCT-ND"
 			(at 124.46 152.4 0)
 			(hide yes)
@@
 			)
 		)
-		(property "Mouser" "771-2N7002PS-115"
+		(property "Mouser" "863-NTJD5121NT1G"
 			(at 124.46 154.94 0)
 			(hide yes)
@@
 			)
 		)
-		(property "TME" "2N7002PS.115"
+		(property "TME" "NTJD5121NT1G"
 			(at 124.46 157.48 0)
 			(hide yes)
@@
 			)
 		)
-		(property "LCSC" "C551419"
+		(property "LCSC" "C15215"
 			(at 124.46 142.24 0)
 			(hide yes)
@@
 			)
 		)
-		(property "Value" "2N7002PS,115"
+		(property "Value" "NTJD5121NT1G"
 			(at 153.67 142.24 0)
 			(hide yes)
@@
 			)
 		)
-		(property "DigiKey" "1727-4791-2-ND"
+		(property "DigiKey" "NTJD5121NT1GOSCT-ND"
 			(at 160.02 152.4 0)
 			(hide yes)
@@
 			)
 		)
-		(property "Mouser" "771-2N7002PS-115"
+		(property "Mouser" "863-NTJD5121NT1G"
 			(at 160.02 154.94 0)
 			(hide yes)
@@
 			)
 		)
-		(property "TME" "2N7002PS.115"
+		(property "TME" "NTJD5121NT1G"
 			(at 160.02 157.48 0)
 			(hide yes)
@@
 			)
 		)
-		(property "LCSC" "C551419"
+		(property "LCSC" "C15215"
 			(at 160.02 142.24 0)
 			(hide yes)
@@
 			)
 		)
-		(property "Value" "2N7002PS,115"
+		(property "Value" "NTJD5121NT1G"
 			(at 66.04 144.145 0)
 			(show_name no)
@@
 			)
 		)
-		(property "DigiKey" "1727-4791-2-ND"
+		(property "DigiKey" "NTJD5121NT1GOSCT-ND"
 			(at 71.12 152.4 0)
 			(hide yes)
@@
 			)
 		)
-		(property "Mouser" "771-2N7002PS-115"
+		(property "Mouser" "863-NTJD5121NT1G"
 			(at 71.12 154.94 0)
 			(hide yes)
@@
 			)
 		)
-		(property "TME" "2N7002PS.115"
+		(property "TME" "NTJD5121NT1G"
 			(at 71.12 157.48 0)
 			(hide yes)
@@
 			)
 		)
-		(property "LCSC" "C551419"
+		(property "LCSC" "C15215"
 			(at 71.12 142.24 0)
 			(hide yes)
