File: KiCad/Digital_inputs.kicad_sch (KiCad schematic)
At the start: 49 parts, among them IC22 TL431B, Q10 NTJD5121NT1G, Q11 NTJD5121NT1G, Q7 NTJD5121NT1G, Q8 NTJD5121NT1G, Q9 NTJD5121NT1G

Commit message: #4
Parts:
- renumbered C95 to C80, C96 to C81, C97 to C82, C98 to C83, C99 to C84, C100 to C85, C101 to C86, C102 to C87, C103 to C88, C104 to C89, C105 to C90, C106 to C91, R43 to R44, R44 to R45, R45 to R46, R46 to R47, R47 to R48, R48 to R49, R49 to R50, R50 to R51, R51 to R52, R52 to R53, R53 to R54, R54 to R55, R55 to R56, R56 to R57, R57 to R58, R58 to R59, R59 to R60, R60 to R61, R61 to R62, R62 to R63, R63 to R64, R64 to R65, R65 to R66, R66 to R67, R67 to R68, R68 to R69, R69 to R70
