File: KiCad/MCU.kicad_sch (KiCad schematic)
At the start: 38 parts, among them IC6 STM32F446ZET6, IC7 W9812G6KH-6, Y1 LF XTAL026392

Commit message: Gerber files added
Parts:
- C25, C27: DigiKey (none) -> 490-12738-1-ND; LCSC (none) -> C77047; Mouser (none) -> 81-GRM188R61E225KA2D; TME (none) -> GRM188R61E225KA12D
- C34, C35: DigiKey (none) -> 1276-1069-1-ND; LCSC (none) -> C1634; Mouser (none) -> 187-CL10C100CB8NNNC; TME (none) -> VJ0603A100JXACW1BC
- FB1: LCSC (none) -> C337877
- R10: DigiKey (none) -> 13-RC0603FR-134K7LTR-ND; LCSC (none) -> C23162; Mouser (none) -> 603-RC0603FR-134K7L; TME (none) -> SMD0603-4K7-1%
Changed lines of the file:
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@@
 			)
 		)
+		(property "LCSC" "C337877"
+			(at 66.04 162.56 0)
+			(hide yes)
+			(show_name no)
+			(do_not_autoplace no)
+			(effects
+				(font
+					(size 0.889 0.889)
+				)
+			)
+		)
 		(pin "1"
 		)
@@
 			)
 		)
-		(property "DigiKey" ""
+		(property "DigiKey" "490-12738-1-ND"
 			(at 129.54 187.96 0)
 			(hide yes)
@@
 			)
 		)
-		(property "Mouser" ""
+		(property "Mouser" "81-GRM188R61E225KA2D"
 			(at 129.54 187.96 0)
 			(hide yes)
@@
 			)
 		)
-		(property "TME" ""
+		(property "TME" "GRM188R61E225KA12D"
 			(at 129.54 187.96 0)
 			(hide yes)
@@
 			)
 		)
-		(property "LCSC" ""
+		(property "LCSC" "C77047"
 			(at 129.54 187.96 0)
 			(hide yes)
@@
 			)
 		)
-		(property "DigiKey" ""
+		(property "DigiKey" "490-12738-1-ND"
 			(at 124.46 187.96 0)
 			(hide yes)
@@
 			)
 		)
-		(property "Mouser" ""
+		(property "Mouser" "81-GRM188R61E225KA2D"
 			(at 124.46 187.96 0)
 			(hide yes)
@@
 			)
 		)
-		(property "TME" ""
+		(property "TME" "GRM188R61E225KA12D"
 			(at 124.46 187.96 0)
 			(hide yes)
@@
 			)
 		)
-		(property "LCSC" ""
+		(property "LCSC" "C77047"
 			(at 124.46 187.96 0)
 			(hide yes)
@@
 			)
 		)
-		(property "TME" ""
+		(property "TME" "VJ0603A100JXACW1BC"
 			(at 190.5 71.12 0)
 			(hide yes)
@@
 			)
 		)
-		(property "DigiKey" ""
+		(property "DigiKey" "1276-1069-1-ND"
 			(at 190.5 71.12 0)
 			(hide yes)
@@
 			)
 		)
-		(property "Mouser" ""
+		(property "Mouser" "187-CL10C100CB8NNNC"
 			(at 190.5 71.12 0)
 			(hide yes)
@@
 			)
 		)
-		(property "LCSC" ""
+		(property "LCSC" "C1634"
 			(at 190.5 71.12 0)
 			(hide yes)
@@
 			)
 		)
-		(property "DigiKey" ""
+		(property "DigiKey" "13-RC0603FR-134K7LTR-ND"
 			(at 175.26 96.52 0)
 			(hide yes)
@@
 			)
 		)
-		(property "Mouser" ""
+		(property "Mouser" "603-RC0603FR-134K7L"
 			(at 175.26 96.52 0)
 			(hide yes)
@@
 			)
 		)
-		(property "TME" ""
+		(property "TME" "SMD0603-4K7-1% "
 			(at 175.26 96.52 0)
 			(hide yes)
@@
 			)
 		)
-		(property "LCSC" ""
+		(property "LCSC" "C23162"
 			(at 175.26 96.52 0)
 			(hide yes)
@@
 			)
 		)
-		(property "TME" ""
+		(property "TME" "VJ0603A100JXACW1BC"
 			(at 190.5 81.28 0)
 			(hide yes)
@@
 			)
 		)
-		(property "DigiKey" ""
+		(property "DigiKey" "1276-1069-1-ND"
 			(at 190.5 81.28 0)
 			(hide yes)
@@
 			)
 		)
-		(property "Mouser" ""
+		(property "Mouser" "187-CL10C100CB8NNNC"
 			(at 190.5 81.28 0)
 			(hide yes)
@@
 			)
 		)
-		(property "LCSC" ""
+		(property "LCSC" "C1634"
 			(at 190.5 81.28 0)
 			(hide yes)

Commit message: BOM update
Parts:
- IC7: value W9812G6KH-6 -> IS42S16400N-6TL; DigiKey W9812G6KH-6-ND -> 1450-1260-ND; LCSC (none) -> C62379; Mouser 454-W9812G6KH-6 -> 822-IM6416SDBATG-6I
- R7: DigiKey (none) -> 13-RC0603FR-1347RLCT-ND; LCSC (none) -> C4328334; Mouser (none) -> 603-RC0603FR-1347RL; TME (none) -> SMD0603-47R-1%
- R8: DigiKey (none) -> 118-CHP0603QFW-1R00ELFCT-ND; LCSC (none) -> C163871; Mouser (none) -> 279-CRG0603F1R0; TME (none) -> SMD0603-1R-1%
Other:
- note added: "SDRAM (64kbit, 4MBx16)"
- note removed: "SDRAM"
Changed lines of the file:
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@@
 	(title_block
 		(title "${project_name}")
-		(date "2026-07-24")
+		(date "2026-07-25")
 		(rev "${project_version}")
 		(company "${project_creator}")
@@
 		)
 	)
-	(text "SDRAM"
+	(text "SDRAM (64kbit, 4MBx16)"
 		(exclude_from_sim no)
 		(at 210.82 17.78 0)
@@
 			)
 		)
-		(property "Value" "W9812G6KH-6"
+		(property "Value" "IS42S16400N-6TL"
 			(at 231.14 119.38 0)
 			(show_name no)
@@
 			)
 		)
-		(property "DigiKey" "W9812G6KH-6-ND"
+		(property "DigiKey" "1450-1260-ND"
 			(at 243.84 71.12 0)
 			(hide yes)
@@
 			)
 		)
-		(property "Mouser" "454-W9812G6KH-6"
+		(property "Mouser" "822-IM6416SDBATG-6I"
 			(at 243.84 71.12 0)
 			(hide yes)
@@
 			)
 		)
+		(property "LCSC" "C62379"
+			(at 243.84 71.12 0)
+			(hide yes)
+			(show_name no)
+			(do_not_autoplace no)
+			(effects
+				(font
+					(size 0.889 0.889)
+				)
+			)
+		)
 		(pin "14"
 		)
@@
 			)
 		)
-		(property "DigiKey" ""
+		(property "DigiKey" "118-CHP0603QFW-1R00ELFCT-ND"
 			(at 139.7 132.08 0)
 			(hide yes)
@@
 			)
 		)
-		(property "Mouser" ""
+		(property "Mouser" "279-CRG0603F1R0"
 			(at 139.7 132.08 0)
 			(hide yes)
@@
 			)
 		)
-		(property "TME" ""
+		(property "TME" "SMD0603-1R-1%"
 			(at 139.7 132.08 0)
 			(hide yes)
@@
 			)
 		)
-		(property "LCSC" ""
+		(property "LCSC" "C163871"
 			(at 139.7 132.08 0)
 			(hide yes)
@@
 			)
 		)
-		(property "DigiKey" ""
+		(property "DigiKey" "13-RC0603FR-1347RLCT-ND"
 			(at 83.82 175.26 0)
 			(hide yes)
@@
 			)
 		)
-		(property "Mouser" ""
+		(property "Mouser" "603-RC0603FR-1347RL"
 			(at 83.82 175.26 0)
 			(hide yes)
@@
 			)
 		)
-		(property "TME" ""
+		(property "TME" "SMD0603-47R-1%"
 			(at 83.82 175.26 0)
 			(hide yes)
@@
 			)
 		)
-		(property "LCSC" ""
+		(property "LCSC" "C4328334"
 			(at 83.82 175.26 0)
 			(hide yes)

Commit message: Y1 value updated
Parts:
- Y1: value LF XTAL026392 -> ABM8-16.000MHZ-10-D7G-T; DigiKey 1923-1009-ND -> 535-14383-1-ND; LCSC C2450580 -> C1986769; Mouser 449-LFXTAL026392BULK -> 815-ABM816.MHZ10D7GT; TME 16.00M-12SM -> CX3225FB16000F0FZZ
Changed lines of the file:
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@@
 			)
 		)
-		(property "Value" "LF XTAL026392"
+		(property "Value" "ABM8-16.000MHZ-10-D7G-T"
 			(at 186.055 78.105 90)
 			(show_name no)
@@
 			)
 		)
-		(property "DigiKey" "1923-1009-ND"
+		(property "DigiKey" "535-14383-1-ND"
 			(at 175.26 76.2 0)
 			(hide yes)
-			(show_name yes)
+			(show_name no)
 			(do_not_autoplace no)
 			(effects
@@
 			)
 		)
-		(property "Mouser" "449-LFXTAL026392BULK"
+		(property "Mouser" "815-ABM816.MHZ10D7GT"
 			(at 172.72 76.2 0)
 			(hide yes)
-			(show_name yes)
+			(show_name no)
 			(do_not_autoplace no)
 			(effects
@@
 			)
 		)
-		(property "TME" "16.00M-12SM"
+		(property "TME" "CX3225FB16000F0FZZ"
 			(at 170.18 73.66 0)
 			(hide yes)
-			(show_name yes)
+			(show_name no)
 			(do_not_autoplace no)
 			(effects
@@
 			)
 		)
-		(property "LCSC" "C2450580"
+		(property "LCSC" "C1986769"
 			(at 182.88 76.2 0)
 			(hide yes)

Commit message: BOM update
Parts:
- R8: Mouser 279-CRG0603F1R0 -> 652-CR0603-F/1R00ELF
Changed lines of the file:
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@@
 	(title_block
 		(title "${project_name}")
-		(date "2026-08-07")
+		(date "2026-08-23")
 		(rev "${project_version}")
 		(company "${project_creator}")
@@
 			)
 		)
-		(property "Mouser" "279-CRG0603F1R0"
+		(property "Mouser" "652-CR0603-F/1R00ELF"
 			(at 139.7 132.08 0)
 			(hide yes)

Commit message: Image of assembled prototype
Parts:
- added LED1: LTST-C170KGKT, PCM_EEZ_SMD:LED_LTST-C170KGKT_LTO-L, symbol PCM_EEZ_discretes:DIODE_LED
- added R70: 750R, PCM_EEZ_passives:R_0603_1608Metric, symbol PCM_EEZ_passives:R-EU
- C16: value 1u -> 1u/50V
- C26: value 4u7 -> 4u7/35V; DigiKey 1276-1044-1-ND -> 1276-6794-1-ND; LCSC C19666 -> C913498; Mouser 187-CL10A475KP8NNNC -> 81-GRM188R6YA475ME5D; TME CL10A475KP8NNNC -> GRM219R6YA475KA73D
Connections:
- net GND: now also LED1.C
- net at IC6.7 (PC13): now also R70.2
- new net: LED1.A, R70.1
- no-connect marks 34 -> 32
