File: KiCad/MCU.kicad_sch (KiCad schematic)
At the start: 40 parts, among them IC6 STM32F446ZET6, IC7 IS42S16400N-6TL, Y1 ABM8-16.000MHZ-10-D7G-T

Commit message: #1
Parts:
- X3: footprint PCM_EEZ_connectors:TC2030 -> PCM_EEZ_connectors:WR-WST_490107670612_DEBUG; symbol PCM_EEZ_connectors:TC2030-IDC -> PCM_EEZ_connectors:WR-WST REDFIT IDC
Other:
- note added: "PCB pads for WR-WST REDFIT IDC"
- note removed: "PCB pads for Tag-Connect TC2030-CTX"
Changed lines of the file:
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@@
 	(title_block
 		(title "${project_name}")
-		(date "2026-09-14")
+		(date "2026-09-19")
 		(rev "${project_version}")
 		(company "${project_creator}")
@@
 		)
 	)
-	(text "PCB pads for\nTag-Connect TC2030-CTX"
+	(text "PCB pads for\nWR-WST REDFIT IDC"
 		(exclude_from_sim no)
 		(at 17.78 139.7 0)
@@
 	)
 	(symbol
-		(lib_id "PCM_EEZ_connectors:TC2030-IDC")
+		(lib_id "PCM_EEZ_connectors:WR-WST REDFIT IDC")
 		(at 45.72 147.32 0)
 		(mirror y)
@@
 		(in_bom no)
 		(on_board yes)
-		(in_pos_files yes)
+		(in_pos_files no)
 		(dnp no)
 		(property "Reference" "X3"
@@
 			)
 		)
-		(property "Footprint" "PCM_EEZ_connectors:TC2030"
-			(at 44.45 165.1 0)
+		(property "Footprint" "PCM_EEZ_connectors:WR-WST_490107670612_DEBUG"
+			(at 45.72 165.1 0)
 			(hide yes)
 			(show_name no)
@@
 			)
 		)
-		(property "Description" "Tag-Connect Plug-of-Nails connector"
-			(at 40.64 165.1 0)
+		(property "Description" "SKEDD 2.54mm Pitch 6 Pin"
+			(at 45.72 167.64 0)
 			(hide yes)
 			(show_name no)

Commit message: DIB_SYNC added to isolator (currently not used)
Connections:
- net DIB_OE_SYNC renamed DIB_SYNC
- no-connect marks 32 -> 33
Changed lines of the file:
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@@
 	(title_block
 		(title "${project_name}")
-		(date "2026-09-19")
+		(date "2026-09-21")
 		(rev "${project_version}")
 		(company "${project_creator}")
@@
 	)
 	(no_connect
+		(at 58.42 111.76)
+	)
+	(no_connect
 		(at 162.56 55.88)
 	)
@@
 		)
 	)
-	(global_label "DIB_OE_SYNC"
+	(global_label "DIB_SYNC"
 		(shape input)
 		(at 53.34 93.98 180)

Commit message: Gerbers updated
Parts:
- C34, C35, Y1: now not fitted; now left out of the parts list
Connections:
- net RCC_OSC_IN renamed CLK_IN
- net RCC_OSC_OUT: no longer names the net of C35.2, IC6.24 (PH1-OSC_OUT), Y1.3
Changed lines of the file:
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@@
 	(title_block
 		(title "${project_name}")
-		(date "2026-09-21")
+		(date "2026-10-08")
 		(rev "${project_version}")
 		(company "${project_creator}")
@@
 		)
 	)
+	(text_box "Ensure that SPI is selected for the bootloader mode in accordance with the instructions in AN2606."
+		(exclude_from_sim no)
+		(at 59.69 15.24 0)
+		(size 27.94 6.1977)
+		(margins 0.9525 0.9525 0.9525 0.9525)
+		(stroke
+			(width 0)
+			(type solid)
+			(color 255 0 0 1)
+		)
+		(fill
+			(type none)
+		)
+		(effects
+			(font
+				(size 0.889 0.889)
+				(color 255 0 0 1)
+			)
+			(justify left top)
+		)
+	)
 	(junction
 		(at 167.64 83.82)
@@
 	)
 	(junction
+		(at 165.1 73.66)
+		(diameter 0)
+		(color 0 0 0 0)
+	)
+	(junction
 		(at 144.78 147.32)
 		(diameter 0)
@@
 	(wire
 		(pts
-			(xy 170.18 73.66) (xy 162.56 73.66)
+			(xy 177.8 73.66) (xy 165.1 73.66)
 		)
 		(stroke
@@
 	(wire
 		(pts
+			(xy 165.1 71.12) (xy 170.18 71.12)
+		)
+		(stroke
+			(width 0)
+			(type default)
+		)
+	)
+	(wire
+		(pts
 			(xy 198.12 76.2) (xy 195.58 76.2)
 		)
@@
 	(wire
 		(pts
-			(xy 170.18 73.66) (xy 170.18 71.12)
+			(xy 177.8 73.66) (xy 177.8 71.12)
 		)
 		(stroke
@@
 	(wire
 		(pts
+			(xy 165.1 73.66) (xy 162.56 73.66)
+		)
+		(stroke
+			(width 0.1524)
+			(type solid)
+		)
+	)
+	(wire
+		(pts
 			(xy 139.7 137.16) (xy 144.78 137.16)
 		)
@@
 	(wire
 		(pts
+			(xy 165.1 71.12) (xy 165.1 73.66)
+		)
+		(stroke
+			(width 0)
+			(type default)
+		)
+	)
+	(wire
+		(pts
 			(xy 48.26 157.48) (xy 48.26 160.02)
 		)
@@
 	(wire
 		(pts
-			(xy 182.88 81.28) (xy 170.18 81.28)
+			(xy 182.88 81.28) (xy 177.8 81.28)
 		)
 		(stroke
@@
 	(wire
 		(pts
-			(xy 182.88 71.12) (xy 170.18 71.12)
+			(xy 182.88 71.12) (xy 177.8 71.12)
 		)
 		(stroke
@@
 	(wire
 		(pts
-			(xy 170.18 76.2) (xy 170.18 81.28)
+			(xy 177.8 76.2) (xy 177.8 81.28)
 		)
 		(stroke
@@
 	(wire
 		(pts
-			(xy 162.56 76.2) (xy 170.18 76.2)
+			(xy 162.56 76.2) (xy 177.8 76.2)
 		)
 		(stroke
@@
 		)
 	)
-	(label "RCC_OSC_IN"
-		(at 170.18 71.12 0)
-		(effects
-			(font
-				(size 0.889 0.889)
-			)
-			(justify left bottom)
-		)
-	)
 	(label "FMC_A1"
 		(at 218.44 33.02 0)
@@
 		)
 	)
-	(label "RCC_OSC_OUT"
-		(at 170.18 81.28 0)
-		(effects
-			(font
-				(size 0.889 0.889)
-			)
-			(justify left bottom)
-		)
-	)
 	(label "FMC_A4"
 		(at 116.84 83.82 0)
@@
 		)
 	)
+	(global_label "CLK_IN"
+		(shape input)
+		(at 170.18 71.12 0)
+		(fields_autoplaced yes)
+		(effects
+			(font
+				(size 0.889 0.889)
+			)
+			(justify left)
+		)
+		(property "Intersheetrefs" "${INTERSHEET_REFS}"
+			(at 176.7991 71.12 0)
+			(hide yes)
+			(show_name no)
+			(do_not_autoplace no)
+			(effects
+				(font
+					(size 1.27 1.27)
+				)
+				(justify left)
+			)
+		)
+	)
 	(global_label "AFE_SPI_MOSI"
 		(shape output)
@@
 		(body_style 1)
 		(exclude_from_sim no)
-		(in_bom yes)
+		(in_bom no)
 		(on_board yes)
-		(in_pos_files yes)
-		(dnp no)
+		(in_pos_files no)
+		(dnp yes)
 		(property "Reference" "Y1"
 			(at 186.055 76.2 90)
@@
 		(in_bom no)
 		(on_board yes)
-		(in_pos_files yes)
+		(in_pos_files no)
 		(dnp yes)
 		(property "Reference" "LED1"
@@
 		(body_style 1)
 		(exclude_from_sim no)
-		(in_bom yes)
+		(in_bom no)
 		(on_board yes)
-		(in_pos_files yes)
-		(dnp no)
+		(in_pos_files no)
+		(dnp yes)
 		(property "Reference" "C34"
 			(at 190.5 69.215 90)
@@
 		(in_bom no)
 		(on_board yes)
-		(in_pos_files yes)
+		(in_pos_files no)
 		(dnp yes)
 		(property "Reference" "R70"
@@
 		(body_style 1)
 		(exclude_from_sim no)
-		(in_bom yes)
+		(in_bom no)
 		(on_board yes)
-		(in_pos_files yes)
-		(dnp no)
+		(in_pos_files no)
+		(dnp yes)
 		(property "Reference" "C35"
 			(at 190.5 79.375 90)

Commit message: #4
Parts:
- removed C21, C22, C23, C24, C30, C31, C32, C33, C36, C37, C38, C39, C40, C41, C42: 100n, PCM_EEZ_passives:C_0603_1608Metric, symbol PCM_EEZ_passives:C-EU
- removed C27: 2u2, PCM_EEZ_passives:C_0603_1608Metric, symbol PCM_EEZ_passives:C-EU
- removed IC6: STM32F446ZET6, PCM_EEZ_SMD:LQFP-144_20X20MM, symbol PCM_EEZ_STM:STM32F446ZCT6
- removed IC7: IS42S16400N-6TL, PCM_EEZ_SMD:TSOPII-54, symbol PCM_EEZ_ICs:IS42S16400
- removed R7: 47R, PCM_EEZ_passives:R_0603_1608Metric, symbol PCM_EEZ_passives:R-EU
- added IC7: STM32F446RET6TR, PCM_EEZ_SMD:LQFP-64_10x10MM, symbol PCM_EEZ_STM:STM32F446RET6TR
- LED1: now in the parts list
- R8: renamed from R70; value 750R -> 1K; DigiKey (none) -> 13-RC0603FR-131KLCT-ND; LCSC (none) -> C21190; Mouser (none) -> 603-RC0603FR-131KL; TME (none) -> CQ0603-1K-1%
- X3: footprint PCM_EEZ_connectors:WR-WST_490107670612_DEBUG -> PCM_EEZ_connectors:WR-WST_490107670612_DEBUG_pads
- renumbered C34 to C17, C35 to C18, C16 to C19, C17 to C20, C25 to C21, C19 to C22, C20 to C23, C26 to C24, C18 to C25, C28 to C26, C29 to C27, R8 to R11
Connections:
- net +3V3: now also IC7.19 (VDD), IC7.32 (VDD), IC7.48 (VDD), IC7.64 (VDD)
- net AFE_EXT_CLK: now also IC7.41 (PA8)
- net AFE_SPI_MISO: now also IC7.52 (PC11)
- net AFE_SPI_MOSI: now also IC7.53 (PC12)
- net AFE_SPI_SCK: now also IC7.51 (PC10)
- net CLK_IN: now also IC7.5 (PH0-OSC_IN)
- net CS_A0: now also IC7.4 (PC15-OSC32_OUT)
- net CS_A1: now also IC7.3 (PC14-OSC32_IN)
- net CS_A2: now also IC7.2 (PC13)
- net DIB_BOOT0: now also IC7.60 (BOOT0)
- net DIB_CSA: now also IC7.20 (PA4)
- net DIB_MISO: now also IC7.22 (PA6)
- net DIB_MOSI: now also IC7.23 (PA7)
- net DIB_SCK: now also IC7.55 (PB3)
- net DIB_SYNC: now also IC7.61 (PB8)
- net GND: now also IC7.12 (VSSA/VREF-), IC7.18 (VSS), IC7.31 (VSS), IC7.47 (VSS), IC7.63 (VSS)
- net I2C_SCL: now also IC7.58 (PB6)
- net I2C_SDA: now also IC7.59 (PB7)
- net IO_SPI_MISO: now also IC7.35 (PB14)
- net IO_SPI_MOSI: now also IC7.9 (PC1)
- net IO_SPI_SCK: now also IC7.38 (PC7)
- net PWM1: now also IC7.14 (PA0)
- net PWM2: now also IC7.15 (PA1)
- net SWCLK: now also IC7.49 (PA14)
- net SWDIO: now also IC7.46 (PA13)
- net USB_CLK: now also IC7.40 (PC9)
- net USB_OTG_HS_ULPI_CK: now also IC7.21 (PA5)
- net USB_OTG_HS_ULPI_D0: now also IC7.17 (PA3)
- net USB_OTG_HS_ULPI_D1: now also IC7.26 (PB0)
- net USB_OTG_HS_ULPI_D2: now also IC7.27 (PB1)
- net USB_OTG_HS_ULPI_D3: now also IC7.29 (PB10)
- net USB_OTG_HS_ULPI_D4: now also IC7.28 (PB2)
- net USB_OTG_HS_ULPI_D5: now also IC7.33 (PB12)
- net USB_OTG_HS_ULPI_D6: now also IC7.34 (PB13)
- net USB_OTG_HS_ULPI_D7: now also IC7.57 (PB5)
- net USB_OTG_HS_ULPI_DIR: now also IC7.10 (PC2)
- net USB_OTG_HS_ULPI_NXT: now also IC7.11 (PC3)
- net USB_OTG_HS_ULPI_STP: now also IC7.8 (PC0)
- net USB_RESET: now also IC7.16 (PA2)
- net ~{AFE_DRDY}: now also IC7.62 (PB9)
- net ~{DIB_FAULT}: now also IC7.25 (PC5)
- net ~{DIB_IRQ}: now also IC7.24 (PC4)
- net ~{DIB_RESET}: now also IC7.7 (NRST)
- net ~{IOEXP1_INT}: now also IC7.44 (PA11)
- net ~{IOEXP2_INT}: now also IC7.45 (PA12)
- net ~{IO_RESET}: now also IC7.54 (PD2)
- net at C18.2, Y1.3: now also IC7.6 (PH1)
- net at C19.1, C20.1, FB1.1: now also IC7.13 (VDDA/VREF+)
- net at C25.2, JP1.2: now also IC7.1 (VBAT)
- net at R8.2: now also IC7.50 (PA15)
- net at C21.2: now also IC7.30 (VCAP)
- new net DIB_TOUT: IC7.39 (PC8)
- new net UART_RX: IC7.43 (PA10)
- new net UART_TX: IC7.42 (PA9)
- no-connect marks 33 -> 5
Other:
- note removed: "Consumption: +3.3 V, up to 110 mA"
- note removed: "IMPORTANT: For PCB layout consult ST AN4661 section 8.4.2"
- note removed: "SDRAM (64kbit, 4MBx16)"
- moved on the sheet: C17, C18, C19, C20, C21, C22, C23, C24, C25, C26, C27, D1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
