File: KiCad/Voltage_current_DACs.kicad_sch (KiCad schematic)
At the start: 39 parts, among them IC13 OPA2196IDR, IC14 DAC7760IPWPR, IC15 DAC7760IPWPR, X4 1844824

Commit message: Gerber files added
Parts:
- C79, C80: DigiKey (none) -> 1276-1018-2-ND; Mouser (none) -> 187-CL10B102KB8NNNC; TME (none) -> CL10B102KB8NNNC
- FB4, FB5: LCSC (none) -> C337877
Changed lines of the file:
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@@
 			)
 		)
-		(property "DigiKey" ""
+		(property "DigiKey" "1276-1018-2-ND"
 			(at 264.16 45.72 0)
 			(hide yes)
@@
 			)
 		)
-		(property "Mouser" ""
+		(property "Mouser" "187-CL10B102KB8NNNC "
 			(at 264.16 45.72 0)
 			(hide yes)
@@
 			)
 		)
-		(property "TME" ""
+		(property "TME" "CL10B102KB8NNNC"
 			(at 264.16 45.72 0)
 			(hide yes)
@@
 			)
 		)
+		(property "LCSC" "C337877"
+			(at 236.22 114.3 90)
+			(hide yes)
+			(show_name no)
+			(do_not_autoplace no)
+			(effects
+				(font
+					(size 0.889 0.889)
+				)
+			)
+		)
 		(pin "1"
 		)
@@
 			)
 		)
+		(property "LCSC" "C337877"
+			(at 236.22 40.64 90)
+			(hide yes)
+			(show_name no)
+			(do_not_autoplace no)
+			(effects
+				(font
+					(size 0.889 0.889)
+				)
+			)
+		)
 		(pin "2"
 		)
@@
 			)
 		)
-		(property "DigiKey" ""
+		(property "DigiKey" "1276-1018-2-ND"
 			(at 264.16 119.38 0)
 			(hide yes)
@@
 			)
 		)
-		(property "Mouser" ""
+		(property "Mouser" "187-CL10B102KB8NNNC "
 			(at 264.16 119.38 0)
 			(hide yes)
@@
 			)
 		)
-		(property "TME" ""
+		(property "TME" "CL10B102KB8NNNC"
 			(at 264.16 119.38 0)
 			(hide yes)

Commit message: BOM update
Parts:
- C69, C71: DigiKey (none) -> 490-4931-1-ND; LCSC (none) -> C161225; Mouser (none) -> 81-GCM188R71H222K37D; TME (none) -> GCM188R71H222KA37D
- C77, C78: DigiKey (none) -> 490-4933-1-ND; LCSC (none) -> C161226; Mouser (none) -> 81-GCM188R71H223KA7J; TME (none) -> GCM188R71H223KA37D
- C79, C80: LCSC (none) -> C1588
- IC13: DigiKey 296-1282-1-ND -> 296-48159-1-ND; LCSC (none) -> C2057972; Mouser 595-TL072CDR -> 595-OPA2196IDR; TME TL072CD-ST -> OPA2196IDR
- IC14, IC15: LCSC (none) -> C2651670
- R23, R24: now left out of the parts list
- R25, R26, R27, R28: DigiKey (none) -> 13-AC0603FR-0715RLCT-ND; LCSC (none) -> C144698; Mouser (none) -> 603-AC0603FR-0715RL; TME (none) -> CQ0603-15R-1%
- TVS1, TVS2: LCSC (none) -> C38558

Commit message: Updated BOM, obsolete parts have been replaced with newer ones
Parts:
- TVS1, TVS2: value PESD12VL1BA,115 -> PESD12VL1BA; DigiKey 1727-3808-1-ND -> 4518-PESD12VL1BACT-ND; Mouser 771-PESD12VL1BA-T/R -> 771-PESD12VS1UAF; TME PESD12VL1BA.115 -> PESD12VL1BA,115
Changed lines of the file:
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@@
 			)
 		)
-		(property "Value" "PESD12VL1BA,115"
+		(property "Value" "PESD12VL1BA"
 			(at 254.508 48.641 90)
 			(show_name no)
@@
 			)
 		)
-		(property "DigiKey" "1727-3808-1-ND"
+		(property "DigiKey" "4518-PESD12VL1BACT-ND"
 			(at 261.62 43.18 0)
 			(hide yes)
@@
 			)
 		)
-		(property "Mouser" "771-PESD12VL1BA-T/R"
+		(property "Mouser" "771-PESD12VS1UAF"
 			(at 264.16 43.18 0)
 			(hide yes)
@@
 			)
 		)
-		(property "TME" "PESD12VL1BA.115"
+		(property "TME" "PESD12VL1BA,115"
 			(at 266.7 43.18 0)
 			(hide yes)
@@
 			)
 		)
-		(property "Value" "PESD12VL1BA,115"
+		(property "Value" "PESD12VL1BA"
 			(at 254.508 122.301 90)
 			(show_name no)
@@
 			)
 		)
-		(property "DigiKey" "1727-3808-1-ND"
+		(property "DigiKey" "4518-PESD12VL1BACT-ND"
 			(at 261.62 116.84 0)
 			(hide yes)
@@
 			)
 		)
-		(property "Mouser" "771-PESD12VL1BA-T/R"
+		(property "Mouser" "771-PESD12VS1UAF"
 			(at 264.16 116.84 0)
 			(hide yes)
@@
 			)
 		)
-		(property "TME" "PESD12VL1BA.115"
+		(property "TME" "PESD12VL1BA,115"
 			(at 266.7 116.84 0)
 			(hide yes)

Commit message: BOM update
Parts:
- D15: now not fitted; now left out of the parts list
- TVS1, TVS2: value PESD12VL1BA -> SD12C-7; DigiKey 4518-PESD12VL1BACT-ND -> 31-SD12C-7CT-ND; LCSC C38558 -> C1977377; Mouser 771-PESD12VS1UAF -> 621-SD12C-7; TME PESD12VL1BA,115 -> SD12C-7
Changed lines of the file:
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@@
 	(title_block
 		(title "${project_name}")
-		(date "2026-08-07")
+		(date "2026-08-23")
 		(rev "${project_version}")
 		(company "${project_creator}")
@@
 		(body_style 1)
 		(exclude_from_sim no)
-		(in_bom yes)
+		(in_bom no)
 		(on_board yes)
 		(in_pos_files yes)
-		(dnp no)
+		(dnp yes)
 		(fields_autoplaced yes)
 		(property "Reference" "D15"
@@
 			)
 		)
-		(property "Value" "PESD12VL1BA"
+		(property "Value" "SD12C-7"
 			(at 254.508 48.641 90)
 			(show_name no)
@@
 			)
 		)
-		(property "DigiKey" "4518-PESD12VL1BACT-ND"
+		(property "DigiKey" "31-SD12C-7CT-ND"
 			(at 261.62 43.18 0)
 			(hide yes)
@@
 			)
 		)
-		(property "Mouser" "771-PESD12VS1UAF"
+		(property "Mouser" "621-SD12C-7"
 			(at 264.16 43.18 0)
 			(hide yes)
@@
 			)
 		)
-		(property "TME" "PESD12VL1BA,115"
+		(property "TME" "SD12C-7"
 			(at 266.7 43.18 0)
 			(hide yes)
@@
 			)
 		)
-		(property "LCSC" "C38558"
+		(property "LCSC" "C1977377"
 			(at 256.54 43.18 90)
 			(hide yes)
@@
 			)
 		)
-		(property "Value" "PESD12VL1BA"
+		(property "Value" "SD12C-7"
 			(at 254.508 122.301 90)
 			(show_name no)
@@
 			)
 		)
-		(property "DigiKey" "4518-PESD12VL1BACT-ND"
+		(property "DigiKey" "31-SD12C-7CT-ND"
 			(at 261.62 116.84 0)
 			(hide yes)
@@
 			)
 		)
-		(property "Mouser" "771-PESD12VS1UAF"
+		(property "Mouser" "621-SD12C-7"
 			(at 264.16 116.84 0)
 			(hide yes)
@@
 			)
 		)
-		(property "TME" "PESD12VL1BA,115"
+		(property "TME" "SD12C-7"
 			(at 266.7 116.84 0)
 			(hide yes)
@@
 			)
 		)
-		(property "LCSC" "C38558"
+		(property "LCSC" "C1977377"
 			(at 256.54 116.84 90)
 			(hide yes)
@@
 		(body_style 1)
 		(exclude_from_sim no)
-		(in_bom yes)
+		(in_bom no)
 		(on_board yes)
 		(in_pos_files yes)
-		(dnp no)
+		(dnp yes)
 		(fields_autoplaced yes)
 		(property "Reference" "D15"

Commit message: Image of assembled prototype
Parts:
- C65, C66, C74, C76: value 4u7 -> 4u7/35V; DigiKey 1276-1044-1-ND -> 1276-6794-1-ND; LCSC C19666 -> C913498; Mouser 187-CL10A475KP8NNNC -> 81-GRM188R6YA475ME5D; TME CL10A475KP8NNNC -> GRM219R6YA475KA73D
Changed lines of the file:
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@@
 	(title_block
 		(title "${project_name}")
-		(date "2026-08-25")
+		(date "2026-08-30")
 		(rev "${project_version}")
 		(company "${project_creator}")
@@
 			)
 		)
-		(property "Value" "4u7"
+		(property "Value" "4u7/35V"
 			(at 162.56 154.305 90)
 			(show_name no)
@@
 			)
 		)
-		(property "DigiKey" "1276-1044-1-ND"
+		(property "DigiKey" "1276-6794-1-ND"
 			(at 162.56 152.4 0)
 			(hide yes)
@@
 			)
 		)
-		(property "Mouser" "187-CL10A475KP8NNNC"
+		(property "Mouser" "81-GRM188R6YA475ME5D"
 			(at 162.56 152.4 0)
 			(hide yes)
@@
 			)
 		)
-		(property "TME" "CL10A475KP8NNNC"
+		(property "TME" "GRM219R6YA475KA73D"
 			(at 162.56 152.4 0)
 			(hide yes)
@@
 			)
 		)
-		(property "LCSC" "C19666"
+		(property "LCSC" "C913498"
 			(at 162.56 152.4 90)
 			(hide yes)
@@
 			)
 		)
-		(property "Value" "4u7"
+		(property "Value" "4u7/35V"
 			(at 175.26 80.645 90)
 			(show_name no)
@@
 			)
 		)
-		(property "DigiKey" "1276-1044-1-ND"
+		(property "DigiKey" "1276-6794-1-ND"
 			(at 175.26 78.74 0)
 			(hide yes)
@@
 			)
 		)
-		(property "Mouser" "187-CL10A475KP8NNNC"
+		(property "Mouser" "81-GRM188R6YA475ME5D"
 			(at 175.26 78.74 0)
 			(hide yes)
@@
 			)
 		)
-		(property "TME" "CL10A475KP8NNNC"
+		(property "TME" "GRM219R6YA475KA73D"
 			(at 175.26 78.74 0)
 			(hide yes)
@@
 			)
 		)
-		(property "LCSC" "C19666"
+		(property "LCSC" "C913498"
 			(at 175.26 78.74 90)
 			(hide yes)
@@
 			)
 		)
-		(property "Value" "4u7"
+		(property "Value" "4u7/35V"
 			(at 162.56 80.645 90)
 			(show_name no)
@@
 			)
 		)
-		(property "DigiKey" "1276-1044-1-ND"
+		(property "DigiKey" "1276-6794-1-ND"
 			(at 162.56 78.74 0)
 			(hide yes)
@@
 			)
 		)
-		(property "Mouser" "187-CL10A475KP8NNNC"
+		(property "Mouser" "81-GRM188R6YA475ME5D"
 			(at 162.56 78.74 0)
 			(hide yes)
@@
 			)
 		)
-		(property "TME" "CL10A475KP8NNNC"
+		(property "TME" "GRM219R6YA475KA73D"
 			(at 162.56 78.74 0)
 			(hide yes)
@@
 			)
 		)
-		(property "LCSC" "C19666"
+		(property "LCSC" "C913498"
 			(at 162.56 78.74 90)
 			(hide yes)
@@
 			)
 		)
-		(property "Value" "4u7"
+		(property "Value" "4u7/35V"
 			(at 175.26 154.305 90)
 			(show_name no)
@@
 			)
 		)
-		(property "DigiKey" "1276-1044-1-ND"
+		(property "DigiKey" "1276-6794-1-ND"
 			(at 175.26 152.4 0)
 			(hide yes)
@@
 			)
 		)
-		(property "Mouser" "187-CL10A475KP8NNNC"
+		(property "Mouser" "81-GRM188R6YA475ME5D"
 			(at 175.26 152.4 0)
 			(hide yes)
@@
 			)
 		)
-		(property "TME" "CL10A475KP8NNNC"
+		(property "TME" "GRM219R6YA475KA73D"
 			(at 175.26 152.4 0)
 			(hide yes)
@@
 			)
 		)
-		(property "LCSC" "C19666"
+		(property "LCSC" "C913498"
 			(at 175.26 152.4 90)
 			(hide yes)
