File: KiCad/Voltage_current_DACs.kicad_sch (KiCad schematic)
At the start: 39 parts, among them IC13 OPA2196IDR, IC14 DAC7760IPWPR, IC15 DAC7760IPWPR, X4 1844824

Commit message: #4
Parts:
- renumbered C61 to C46, C62 to C47, C63 to C48, C64 to C49, C65 to C50, C66 to C51, C67 to C52, C68 to C53, C69 to C54, C70 to C55, C71 to C56, C72 to C57, C73 to C58, C74 to C59, C75 to C60, C76 to C61, C77 to C62, C78 to C63, C79 to C64, C80 to C65, R22 to R23, R23 to R24, R24 to R25, R25 to R26, R26 to R27, R27 to R28, R28 to R29, TP5 to TP6, TP6 to TP7
Changed lines of the file:
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@@
 	(title_block
 		(title "${project_name}")
-		(date "2026-10-08")
+		(date "2026-10-17")
 		(rev "${project_version}")
 		(company "${project_creator}")
@@
 		(in_pos_files yes)
 		(dnp no)
-		(property "Reference" "C61"
+		(property "Reference" "C46"
 			(at 114.3 149.225 90)
 			(show_name no)
@@
 			(project "EEZ DIB MIO168plus"
 				(path "/8165d74e-be16-4c9d-8240-91910dc4b43e/bf314781-ba18-468c-bf18-9e97e69917dd"
-					(reference "C61")
+					(reference "C46")
 					(unit 1)
 				)
@@
 		(in_pos_files yes)
 		(dnp no)
-		(property "Reference" "C69"
+		(property "Reference" "C54"
 			(at 172.72 40.005 90)
 			(show_name no)
@@
 			(project "EEZ DIB MIO168plus"
 				(path "/8165d74e-be16-4c9d-8240-91910dc4b43e/bf314781-ba18-468c-bf18-9e97e69917dd"
-					(reference "C69")
+					(reference "C54")
 					(unit 1)
 				)
@@
 		(in_pos_files yes)
 		(dnp no)
-		(property "Reference" "C75"
+		(property "Reference" "C60"
 			(at 175.26 132.08 0)
 			(show_name no)
@@
 			(project "EEZ DIB MIO168plus"
 				(path "/8165d74e-be16-4c9d-8240-91910dc4b43e/bf314781-ba18-468c-bf18-9e97e69917dd"
-					(reference "C75")
+					(reference "C60")
 					(unit 1)
 				)
@@
 		(in_pos_files yes)
 		(dnp no)
-		(property "Reference" "C79"
+		(property "Reference" "C64"
 			(at 264.16 45.72 0)
 			(show_name no)
@@
 			(project "EEZ DIB MIO168plus"
 				(path "/8165d74e-be16-4c9d-8240-91910dc4b43e/bf314781-ba18-468c-bf18-9e97e69917dd"
-					(reference "C79")
+					(reference "C64")
 					(unit 1)
 				)
@@
 		(in_pos_files yes)
 		(dnp no)
-		(property "Reference" "C68"
+		(property "Reference" "C53"
 			(at 162.56 146.685 90)
 			(show_name no)
@@
 			(project "EEZ DIB MIO168plus"
 				(path "/8165d74e-be16-4c9d-8240-91910dc4b43e/bf314781-ba18-468c-bf18-9e97e69917dd"
-					(reference "C68")
+					(reference "C53")
 					(unit 1)
 				)
@@
 		(in_pos_files yes)
 		(dnp no)
-		(property "Reference" "C73"
+		(property "Reference" "C58"
 			(at 175.26 58.42 0)
 			(show_name no)
@@
 			(project "EEZ DIB MIO168plus"
 				(path "/8165d74e-be16-4c9d-8240-91910dc4b43e/bf314781-ba18-468c-bf18-9e97e69917dd"
-					(reference "C73")
+					(reference "C58")
 					(unit 1)
 				)
@@
 		(in_pos_files yes)
 		(dnp no)
-		(property "Reference" "R28"
+		(property "Reference" "R29"
 			(at 220.98 118.11 90)
 			(show_name no)
@@
 			(project "EEZ DIB MIO168plus"
 				(path "/8165d74e-be16-4c9d-8240-91910dc4b43e/bf314781-ba18-468c-bf18-9e97e69917dd"
-					(reference "R28")
+					(reference "R29")
 					(unit 1)
 				)
@@
 		(in_pos_files yes)
 		(dnp no)
-		(property "Reference" "C64"
+		(property "Reference" "C49"
 			(at 124.206 129.794 0)
 			(show_name no)
@@
 			(project "EEZ DIB MIO168plus"
 				(path "/8165d74e-be16-4c9d-8240-91910dc4b43e/bf314781-ba18-468c-bf18-9e97e69917dd"
-					(reference "C64")
+					(reference "C49")
 					(unit 1)
 				)
@@
 		(in_pos_files yes)
 		(dnp no)
-		(property "Reference" "C66"
+		(property "Reference" "C51"
 			(at 162.56 151.765 90)
 			(show_name no)
@@
 			(project "EEZ DIB MIO168plus"
 				(path "/8165d74e-be16-4c9d-8240-91910dc4b43e/bf314781-ba18-468c-bf18-9e97e69917dd"
-					(reference "C66")
+					(reference "C51")
 					(unit 1)
 				)
@@
 		(in_pos_files yes)
 		(dnp no)
-		(property "Reference" "C70"
+		(property "Reference" "C55"
 			(at 175.26 73.025 90)
 			(show_name no)
@@
 			(project "EEZ DIB MIO168plus"
 				(path "/8165d74e-be16-4c9d-8240-91910dc4b43e/bf314781-ba18-468c-bf18-9e97e69917dd"
-					(reference "C70")
+					(reference "C55")
 					(unit 1)
 				)
@@
 		(in_pos_files yes)
 		(dnp no)
-		(property "Reference" "R25"
+		(property "Reference" "R26"
 			(at 220.98 26.67 90)
 			(show_name no)
@@
 			(project "EEZ DIB MIO168plus"
 				(path "/8165d74e-be16-4c9d-8240-91910dc4b43e/bf314781-ba18-468c-bf18-9e97e69917dd"
-					(reference "R25")
+					(reference "R26")
 					(unit 1)
 				)
@@
 		(in_pos_files yes)
 		(dnp no)
-		(property "Reference" "C71"
+		(property "Reference" "C56"
 			(at 172.72 113.665 90)
 			(show_name no)
@@
 			(project "EEZ DIB MIO168plus"
 				(path "/8165d74e-be16-4c9d-8240-91910dc4b43e/bf314781-ba18-468c-bf18-9e97e69917dd"
-					(reference "C71")
+					(reference "C56")
 					(unit 1)
 				)
@@
 		(in_pos_files yes)
 		(dnp no)
-		(property "Reference" "C62"
+		(property "Reference" "C47"
 			(at 114.3 164.465 90)
 			(show_name no)
@@
 			(project "EEZ DIB MIO168plus"
 				(path "/8165d74e-be16-4c9d-8240-91910dc4b43e/bf314781-ba18-468c-bf18-9e97e69917dd"
-					(reference "C62")
+					(reference "C47")
 					(unit 1)
 				)
@@
 		(in_pos_files yes)
 		(dnp no)
-		(property "Reference" "R26"
+		(property "Reference" "R27"
 			(at 220.98 44.45 90)
 			(show_name no)
@@
 			(project "EEZ DIB MIO168plus"
 				(path "/8165d74e-be16-4c9d-8240-91910dc4b43e/bf314781-ba18-468c-bf18-9e97e69917dd"
-					(reference "R26")
+					(reference "R27")
 					(unit 1)
 				)
@@
 		(in_pos_files yes)
 		(dnp no)
-		(property "Reference" "R27"
+		(property "Reference" "R28"
 			(at 220.98 100.33 90)
 			(show_name no)
@@
 			(project "EEZ DIB MIO168plus"
 				(path "/8165d74e-be16-4c9d-8240-91910dc4b43e/bf314781-ba18-468c-bf18-9e97e69917dd"
-					(reference "R27")
+					(reference "R28")
 					(unit 1)
 				)
@@
 		(in_pos_files no)
 		(dnp no)
-		(property "Reference" "TP5"
+		(property "Reference" "TP6"
 			(at 250.825 34.29 90)
 			(show_name no)
@@
 			(project "EEZ DIB MIO168plus"
 				(path "/8165d74e-be16-4c9d-8240-91910dc4b43e/bf314781-ba18-468c-bf18-9e97e69917dd"
-					(reference "TP5")
+					(reference "TP6")
 					(unit 1)
 				)
@@
 		(in_pos_files yes)
 		(dnp no)
-		(property "Reference" "C74"
+		(property "Reference" "C59"
 			(at 175.26 78.105 90)
 			(show_name no)
@@
 			(project "EEZ DIB MIO168plus"
 				(path "/8165d74e-be16-4c9d-8240-91910dc4b43e/bf314781-ba18-468c-bf18-9e97e69917dd"
-					(reference "C74")
+					(reference "C59")
 					(unit 1)
 				)
@@
 		(in_pos_files no)
 		(dnp no)
-		(property "Reference" "TP6"
+		(property "Reference" "TP7"
 			(at 250.825 107.95 90)
 			(show_name no)
@@
 			(project "EEZ DIB MIO168plus"
 				(path "/8165d74e-be16-4c9d-8240-91910dc4b43e/bf314781-ba18-468c-bf18-9e97e69917dd"
-					(reference "TP6")
+					(reference "TP7")
 					(unit 1)
 				)
@@
 		(in_pos_files no)
 		(dnp yes)
-		(property "Reference" "R23"
+		(property "Reference" "R24"
 			(at 172.72 31.75 90)
 			(show_name no)
@@
 			(project "EEZ DIB MIO168plus"
 				(path "/8165d74e-be16-4c9d-8240-91910dc4b43e/bf314781-ba18-468c-bf18-9e97e69917dd"
-					(reference "R23")
+					(reference "R24")
 					(unit 1)
 				)
@@
 		(in_pos_files yes)
 		(dnp no)
-		(property "Reference" "C77"
+		(property "Reference" "C62"
 			(at 183.515 53.34 0)
 			(show_name no)
@@
 			(project "EEZ DIB MIO168plus"
 				(path "/8165d74e-be16-4c9d-8240-91910dc4b43e/bf314781-ba18-468c-bf18-9e97e69917dd"
-					(reference "C77")
+					(reference "C62")
 					(unit 1)
 				)
@@
 		(in_pos_files yes)
 		(dnp no)
-		(property "Reference" "C72"
+		(property "Reference" "C57"
 			(at 175.26 146.685 90)
 			(show_name no)
@@
 			(project "EEZ DIB MIO168plus"
 				(path "/8165d74e-be16-4c9d-8240-91910dc4b43e/bf314781-ba18-468c-bf18-9e97e69917dd"
-					(reference "C72")
+					(reference "C57")
 					(unit 1)
 				)
@@
 		(in_pos_files yes)
 		(dnp no)
-		(property "Reference" "C80"
+		(property "Reference" "C65"
 			(at 264.16 119.38 0)
 			(show_name no)
@@
 			(project "EEZ DIB MIO168plus"
 				(path "/8165d74e-be16-4c9d-8240-91910dc4b43e/bf314781-ba18-468c-bf18-9e97e69917dd"
-					(reference "C80")
+					(reference "C65")
 					(unit 1)
 				)
@@
 		(in_pos_files yes)
 		(dnp no)
-		(property "Reference" "C65"
+		(property "Reference" "C50"
 			(at 162.56 78.105 90)
 			(show_name no)
@@
 			(project "EEZ DIB MIO168plus"
 				(path "/8165d74e-be16-4c9d-8240-91910dc4b43e/bf314781-ba18-468c-bf18-9e97e69917dd"
-					(reference "C65")
+					(reference "C50")
 					(unit 1)
 				)
@@
 		(in_pos_files yes)
 		(dnp no)
-		(property "Reference" "C76"
+		(property "Reference" "C61"
 			(at 175.26 151.765 90)
 			(show_name no)
@@
 			(project "EEZ DIB MIO168plus"
 				(path "/8165d74e-be16-4c9d-8240-91910dc4b43e/bf314781-ba18-468c-bf18-9e97e69917dd"
-					(reference "C76")
+					(reference "C61")
 					(unit 1)
 				)
@@
 		(in_pos_files yes)
 		(dnp no)
-		(property "Reference" "C63"
+		(property "Reference" "C48"
 			(at 124.46 55.88 0)
 			(show_name no)
@@
 			(project "EEZ DIB MIO168plus"
 				(path "/8165d74e-be16-4c9d-8240-91910dc4b43e/bf314781-ba18-468c-bf18-9e97e69917dd"
-					(reference "C63")
+					(reference "C48")
 					(unit 1)
 				)
@@
 		(in_pos_files yes)
 		(dnp no)
-		(property "Reference" "C78"
+		(property "Reference" "C63"
 			(at 182.88 127 0)
 			(show_name no)
@@
 			(project "EEZ DIB MIO168plus"
 				(path "/8165d74e-be16-4c9d-8240-91910dc4b43e/bf314781-ba18-468c-bf18-9e97e69917dd"
-					(reference "C78")
+					(reference "C63")
 					(unit 1)
 				)
@@
 		(in_pos_files yes)
 		(dnp no)
-		(property "Reference" "C67"
+		(property "Reference" "C52"
 			(at 162.56 73.025 90)
 			(show_name no)
@@
 			(project "EEZ DIB MIO168plus"
 				(path "/8165d74e-be16-4c9d-8240-91910dc4b43e/bf314781-ba18-468c-bf18-9e97e69917dd"
-					(reference "C67")
+					(reference "C52")
 					(unit 1)
 				)
@@
 		(in_pos_files no)
 		(dnp yes)
-		(property "Reference" "R24"
+		(property "Reference" "R25"
 			(at 172.72 105.41 90)
 			(show_name no)
@@
 			(project "EEZ DIB MIO168plus"
 				(path "/8165d74e-be16-4c9d-8240-91910dc4b43e/bf314781-ba18-468c-bf18-9e97e69917dd"
-					(reference "R24")
+					(reference "R25")
 					(unit 1)
 				)
@@
 		(in_pos_files yes)
 		(dnp no)
-		(property "Reference" "R22"
+		(property "Reference" "R23"
 			(at 101.6 67.31 90)
 			(show_name no)
@@
 			(project "EEZ DIB MIO168plus"
 				(path "/8165d74e-be16-4c9d-8240-91910dc4b43e/bf314781-ba18-468c-bf18-9e97e69917dd"
-					(reference "R22")
+					(reference "R23")
 					(unit 1)
 				)
