File: KiCad/EEZ DIB MIO168plus front mask.kicad_pcb (KiCad board)
At the start: 2 copper layers, 17.2 x 111.5 mm, 3 parts

Commit message: Front mask updated
Other:
- board size 17.2 x 111.5 mm -> 17.6 x 111.5 mm
Changed lines of the file:
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@@
 	(title_block
 		(title "DCP405+ Front mask")
-		(date "2025-10-04")
+		(date "2026-10-16")
 		(rev "r4B2")
 		(company "Envox d.o.o.")
@@
 			(layer "F.SilkS"
 				(type "Top Silk Screen")
+				(color "Black")
 			)
 			(layer "F.Paste"
@@
 			(layer "F.Mask"
 				(type "Top Solder Mask")
+				(color "White")
 				(thickness 0.01)
 			)
@@
 			(layer "dielectric 1"
 				(type "core")
+				(color "Aluminum")
 				(thickness 1.51)
 				(material "FR4")
@@
 			(layer "B.Mask"
 				(type "Bottom Solder Mask")
+				(color "White")
 				(thickness 0.01)
 			)
@@
 			(layer "B.SilkS"
 				(type "Bottom Silk Screen")
+				(color "Black")
 			)
 			(copper_finish "None")
@@
 		(capping no)
 		(filling no)
+		(zone_defaults)
 		(pcbplotparams
-			(layerselection 0x00000000_00000000_55555555_57555577)
+			(layerselection 0x00000000_00000000_55555555_57557573)
 			(plot_on_all_layers_selection 0x00000000_00000000_00000000_00000000)
 			(disableapertmacros no)
@@
 			(at -1.8 0)
 			(size 0.8 0.8)
-			(drill 0.5)
+			(drill 0.6)
 			(layers "*.Cu" "F.Mask")
 			(remove_unused_layers no)
@@
 			(at -1.27 -1.27)
 			(size 0.8 0.8)
-			(drill 0.5)
+			(drill 0.6)
 			(layers "*.Cu" "F.Mask")
 			(remove_unused_layers no)
@@
 			(at -1.27 1.27)
 			(size 0.8 0.8)
-			(drill 0.5)
+			(drill 0.6)
 			(layers "*.Cu" "F.Mask")
 			(remove_unused_layers no)
@@
 			(at 0 -1.8)
 			(size 0.8 0.8)
-			(drill 0.5)
+			(drill 0.6)
 			(layers "*.Cu" "F.Mask")
 			(remove_unused_layers no)
@@
 			(at 0 1.8)
 			(size 0.8 0.8)
-			(drill 0.5)
+			(drill 0.6)
 			(layers "*.Cu" "F.Mask")
 			(remove_unused_layers no)
@@
 			(at 1.27 -1.27)
 			(size 0.8 0.8)
-			(drill 0.5)
+			(drill 0.6)
 			(layers "*.Cu" "F.Mask")
 			(remove_unused_layers no)
@@
 			(at 1.27 1.27)
 			(size 0.8 0.8)
-			(drill 0.5)
+			(drill 0.6)
 			(layers "*.Cu" "F.Mask")
 			(remove_unused_layers no)
@@
 			(at 1.8 0)
 			(size 0.8 0.8)
-			(drill 0.5)
+			(drill 0.6)
 			(layers "*.Cu" "F.Mask")
 			(remove_unused_layers no)
@@
 			(at -1.8 0)
 			(size 0.8 0.8)
-			(drill 0.5)
+			(drill 0.6)
 			(layers "*.Cu" "F.Mask")
 			(remove_unused_layers no)
@@
 			(at -1.27 -1.27)
 			(size 0.8 0.8)
-			(drill 0.5)
+			(drill 0.6)
 			(layers "*.Cu" "F.Mask")
 			(remove_unused_layers no)
@@
 			(at -1.27 1.27)
 			(size 0.8 0.8)
-			(drill 0.5)
+			(drill 0.6)
 			(layers "*.Cu" "F.Mask")
 			(remove_unused_layers no)
@@
 			(at 0 -1.8)
 			(size 0.8 0.8)
-			(drill 0.5)
+			(drill 0.6)
 			(layers "*.Cu" "F.Mask")
 			(remove_unused_layers no)
@@
 			(at 0 1.8)
 			(size 0.8 0.8)
-			(drill 0.5)
+			(drill 0.6)
 			(layers "*.Cu" "F.Mask")
 			(remove_unused_layers no)
@@
 			(at 1.27 -1.27)
 			(size 0.8 0.8)
-			(drill 0.5)
+			(drill 0.6)
 			(layers "*.Cu" "F.Mask")
 			(remove_unused_layers no)
@@
 			(at 1.27 1.27)
 			(size 0.8 0.8)
-			(drill 0.5)
+			(drill 0.6)
 			(layers "*.Cu" "F.Mask")
 			(remove_unused_layers no)
@@
 			(at 1.8 0)
 			(size 0.8 0.8)
-			(drill 0.5)
+			(drill 0.6)
 			(layers "*.Cu" "F.Mask")
 			(remove_unused_layers no)
@@
 	)
 	(gr_rect
-		(start 140.5 144.6)
-		(end 157.95 150.1)
+		(start 140.3 38.5)
+		(end 157.97 44)
 		(stroke
-			(width 0.1)
+			(width 0.05)
 			(type solid)
 		)
@@
 	)
 	(gr_rect
-		(start 140.52 38.5)
-		(end 157.97 44)
+		(start 140.3 144.6)
+		(end 157.95 150.1)
 		(stroke
-			(width 0.1)
+			(width 0.05)
 			(type solid)
 		)
@@
 	)
 	(gr_rect
-		(start 140.5 144.6)
-		(end 157.95 150.1)
+		(start 140.3 38.5)
+		(end 157.95 44)
 		(stroke
-			(width 0.1)
+			(width 0.05)
 			(type solid)
 		)
@@
 	)
 	(gr_rect
-		(start 140.52 38.5)
-		(end 157.97 44)
+		(start 140.3 144.6)
+		(end 157.95 150.1)
 		(stroke
-			(width 0.1)
+			(width 0.05)
 			(type solid)
 		)
@@
 	)
 	(gr_line
-		(start 140.5 150)
-		(end 140.5 38.5)
+		(start 140.3 150)
+		(end 140.3 38.5)
 		(stroke
 			(width 0.05)
@@
 		)
 		(fill no)
+		(locked yes)
 		(layer "Edge.Cuts")
 	)
@@
 		(layer "Edge.Cuts")
 	)
-	(gr_circle
-		(center 149.25 41.75)
-		(end 150.25 41.75)
-		(stroke
-			(width 0.05)
-			(type solid)
-		)
-		(fill no)
-		(locked yes)
-		(layer "Edge.Cuts")
-	)
-	(gr_circle
-		(center 149.25 146.75)
-		(end 150.25 146.75)
-		(stroke
-			(width 0.05)
-			(type solid)
-		)
-		(fill no)
-		(locked yes)
-		(layer "Edge.Cuts")
-	)
 	(gr_line
-		(start 157.75 38.5)
-		(end 140.5 38.5)
+		(start 157.95 38.5)
+		(end 140.3 38.5)
 		(stroke
 			(width 0.05)
@@
 	)
 	(gr_line
-		(start 157.75 38.5)
-		(end 157.75 150)
+		(start 157.95 38.5)
+		(end 157.95 150)
 		(stroke
 			(width 0.05)
@@
 	)
 	(gr_line
-		(start 157.75 150)
-		(end 140.5 150)
+		(start 157.95 150)
+		(end 140.3 150)
 		(stroke
 			(width 0.05)
@@
 			(keep_text_aligned yes)
 		)
-		(gr_text "3307,0866"
+		(gr_text "84"
 			(at 155.65 96 90)
 			(layer "User.1")
@@
 			(keep_text_aligned yes)
 		)
-		(gr_text "127,95"
+		(gr_text "3,25"
 			(at 160.86 40.187499 90)
 			(layer "User.1")
@@
 			(keep_text_aligned yes)
 		)
-		(gr_text "295,3 mils"
+		(gr_text "7,5 mm"
 			(at 144.22 48.342499 0)
 			(layer "User.1")
@@
 			(keep_text_aligned yes)
 		)
-		(gr_text "472,4 mils"
+		(gr_text "12,0 mm"
 			(at 135.93 144 90)
 			(layer "User.1")
@@
 			(keep_text_aligned yes)
 		)
-		(gr_text "407,4803"
+		(gr_text "10,35"
 			(at 152.45 59.175 90)
 			(layer "User.1")
@@
 			(keep_text_aligned yes)
 		)
-		(gr_text "679,1339"
+		(gr_text "17,25"
 			(at 149.125 151.65 0)
 			(layer "User.1")
@@
 			(keep_text_aligned yes)
 		)
-		(gr_text "689,4 mils"
+		(gr_text "17,5 mm"
 			(at 149.255 143.002499 0)
 			(layer "User.1")
@@
 			(keep_text_aligned yes)
 		)
-		(gr_text "1647,6378"
+		(gr_text "41,85"
 			(at 142.4 74.925 90)
 			(layer "User.1")
@@
 			(keep_text_aligned yes)
 		)
-		(gr_text "1240,1575"
+		(gr_text "31,5"
 			(at 154.35 118.45 90)
 			(layer "User.1")
@@
 			(keep_text_aligned yes)
 		)
-		(gr_text "127,9528"
+		(gr_text "3,25"
 			(at 153.1 148.375 90)
 			(layer "User.1")
@@
 			(keep_text_aligned yes)
 		)
-		(gr_text "295,2756"
+		(gr_text "7,5"
 			(at 148.75 96.85 0)
 			(layer "User.1")
@@
 			(keep_text_aligned yes)
 		)
-		(gr_text "681,1024"
+		(gr_text "17,3"
 			(at 132.95 141.35 90)
 			(layer "User.1")
@@
 			(keep_text_aligned yes)
 		)
-		(gr_text "296,1 mils"
+		(gr_text "7,5 mm"
 			(at 144.24 133.002499 0)
 			(layer "User.1")
@@
 			(keep_text_aligned yes)
 		)
-		(gr_text "62,9921"
+		(gr_text "1,6"
 			(at 144.7 145.15 0)
 			(layer "User.2")
@@
 			(keep_text_aligned yes)
 		)
-		(gr_text "133,8583"
+		(gr_text "3,4"
 			(at 142.2 56.35 0)
 			(layer "User.2")
@@
 	)
 	(zone
-		(layer "F.Cu")
+		(layers "F.Cu" "B.Cu")
 		(hatch edge 0.2)
 		(connect_pads
@@
 			)
 		)
-	)
-	(zone
-		(layer "B.Cu")
-		(hatch edge 0.2)
-		(connect_pads
-			(clearance 0.2)
-		)
-		(min_thickness 0.25)
-		(fill yes
-			(thermal_gap 0.5)
-			(thermal_bridge_width 0.5)
-			(island_removal_mode 1)
-		)
-		(polygon
-			(pts
-				(xy 139.330895 37.659318) (xy 158.43498 37.654187) (xy 158.185013 150.869386) (xy 139.810895 150.859318)
-			)
-		)

Commit message: #4
Changed lines of the file:
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@@
 		(capping no)
 		(filling no)
-		(zone_defaults)
 		(pcbplotparams
 			(layerselection 0x00000000_00000000_55555555_57557573)
@@
 			(at -1.8 0)
 			(size 0.8 0.8)
-			(drill 0.6)
+			(drill 0.65)
 			(layers "*.Cu" "F.Mask")
 			(remove_unused_layers no)
@@
 			(at -1.27 -1.27)
 			(size 0.8 0.8)
-			(drill 0.6)
+			(drill 0.65)
 			(layers "*.Cu" "F.Mask")
 			(remove_unused_layers no)
@@
 			(at -1.27 1.27)
 			(size 0.8 0.8)
-			(drill 0.6)
+			(drill 0.65)
 			(layers "*.Cu" "F.Mask")
 			(remove_unused_layers no)
@@
 			(at 0 -1.8)
 			(size 0.8 0.8)
-			(drill 0.6)
+			(drill 0.65)
 			(layers "*.Cu" "F.Mask")
 			(remove_unused_layers no)
@@
 			(at 0 1.8)
 			(size 0.8 0.8)
-			(drill 0.6)
+			(drill 0.65)
 			(layers "*.Cu" "F.Mask")
 			(remove_unused_layers no)
@@
 			(at 1.27 -1.27)
 			(size 0.8 0.8)
-			(drill 0.6)
+			(drill 0.65)
 			(layers "*.Cu" "F.Mask")
 			(remove_unused_layers no)
@@
 			(at 1.27 1.27)
 			(size 0.8 0.8)
-			(drill 0.6)
+			(drill 0.65)
 			(layers "*.Cu" "F.Mask")
 			(remove_unused_layers no)
@@
 			(at 1.8 0)
 			(size 0.8 0.8)
-			(drill 0.6)
+			(drill 0.65)
 			(layers "*.Cu" "F.Mask")
 			(remove_unused_layers no)
@@
 			(at -1.8 0)
 			(size 0.8 0.8)
-			(drill 0.6)
+			(drill 0.65)
 			(layers "*.Cu" "F.Mask")
 			(remove_unused_layers no)
@@
 			(at -1.27 -1.27)
 			(size 0.8 0.8)
-			(drill 0.6)
+			(drill 0.65)
 			(layers "*.Cu" "F.Mask")
 			(remove_unused_layers no)
@@
 			(at -1.27 1.27)
 			(size 0.8 0.8)
-			(drill 0.6)
+			(drill 0.65)
 			(layers "*.Cu" "F.Mask")
 			(remove_unused_layers no)
@@
 			(at 0 -1.8)
 			(size 0.8 0.8)
-			(drill 0.6)
+			(drill 0.65)
 			(layers "*.Cu" "F.Mask")
 			(remove_unused_layers no)
@@
 			(at 0 1.8)
 			(size 0.8 0.8)
-			(drill 0.6)
+			(drill 0.65)
 			(layers "*.Cu" "F.Mask")
 			(remove_unused_layers no)
@@
 			(at 1.27 -1.27)
 			(size 0.8 0.8)
-			(drill 0.6)
+			(drill 0.65)
 			(layers "*.Cu" "F.Mask")
 			(remove_unused_layers no)
@@
 			(at 1.27 1.27)
 			(size 0.8 0.8)
-			(drill 0.6)
+			(drill 0.65)
 			(layers "*.Cu" "F.Mask")
 			(remove_unused_layers no)
@@
 			(at 1.8 0)
 			(size 0.8 0.8)
-			(drill 0.6)
-			(layers "*.Cu" "F.Mask")
-			(remove_unused_layers no)
+			(drill 0.65)
+			(layers "*.Cu" "F.Mask")
+			(remove_unused_layers no)
