File: KiCad/EEZ DIB MIO168plus.kicad_sch (KiCad schematic)
At the start: 12 parts

Commit message: #4
Parts:
- renumbered LOGO7 to LOGO6
Other:
- sheet ADIB, PWM, AFE connectors renamed Isolated power, PWM, Bias power
- sheet MCU, SDRAM renamed MCU
- sheet Isolated power, PWM, Bias power: file ADIB_PWM.kicad_sch -> iso_power.kicad_sch
Changed lines of the file:
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@@
 	(title_block
 		(title "${project_name}")
-		(date "2026-10-08")
+		(date "2026-10-17")
 		(rev "${project_version}")
 		(company "${project_creator}")
@@
 		(dnp no)
 		(fields_autoplaced yes)
-		(property "Reference" "LOGO7"
+		(property "Reference" "LOGO6"
 			(at 68.58 186.0675 0)
 			(hide yes)
@@
 			(project "EEZ DIB MIO168plus"
 				(path "/8165d74e-be16-4c9d-8240-91910dc4b43e"
-					(reference "LOGO7")
+					(reference "LOGO6")
 					(unit 1)
 				)
@@
 			(color 0 0 0 0)
 		)
-		(property "Sheetname" "ADIB, PWM, AFE connectors"
+		(property "Sheetname" "Isolated power, PWM, Bias power"
 			(at 124.46 24.6884 0)
 			(show_name no)
@@
 			)
 		)
-		(property "Sheetfile" "ADIB_PWM.kicad_sch"
+		(property "Sheetfile" "iso_power.kicad_sch"
 			(at 124.46 29.7946 0)
 			(show_name no)
@@
 			(color 0 0 0 0)
 		)
-		(property "Sheetname" "MCU, SDRAM"
+		(property "Sheetname" "MCU"
 			(at 76.2 24.6884 0)
 			(show_name no)
