File: KiCad/iso_power.kicad_sch (KiCad schematic)
At the start: 65 parts, among them IC10 MC78L15ACDR2G, IC11 MC79L15ACDR2G, IC12 74HC126PW,118, IC8 SN6505BDBVT, IC9 TPS7A2033PDBVR, Q1 MMBT5401, Q2 MMBT5551, Q3 MMBT5551, Q4 DMP3099L, Q5 2N7002, Q6 DMP3099L

Commit message: #4
Parts:
- renumbered C43 to C28, C44 to C29, C45 to C30, C46 to C31, C47 to C32, C48 to C33, C49 to C34, C50 to C35, C51 to C36, C52 to C37, C53 to C38, C54 to C39, C55 to C40, C56 to C41, C57 to C42, C58 to C43, C59 to C44, C60 to C45, R11 to R12, R12 to R13, R13 to R14, R14 to R15, R15 to R16, R16 to R17, R17 to R18, R18 to R19, R19 to R20, R20 to R21, R21 to R22, TP1 to TP2, TP2 to TP3, TP3 to TP4, TP4 to TP5
